Commit message: Update inertia, mass, COM

File: xacro/bolt.urdf.xacro (robot description, xacro)
@@ -13,10 +13,14 @@
     <!-- BASE LINK INERTIAL -->
     <inertial>
-        <origin xyz="0 0 0" rpy="0 0 0" />
-        <mass value="0.6"/>
+        <origin xyz="-0.00245656 -0.00078880 0.03308090" rpy="0 0 0" />
+        <mass value="0.61436936"/>
         <!-- The base is extremely symmetrical. -->
-        <inertia ixx="0.00578574" ixy="0.0" ixz="0.0"
-                                  iyy="0.01938108" iyz="0.0"
-                                                   izz="0.02476124"
+        <!--inertia ixx="0.00578574" ixy="0.0" ixz="0.0"
+                 iyy="0.01938108" iyz="0.0"
+                 izz="0.02476124"
+        /-->
+        <inertia ixx="0.00132170" ixy="0.00000117" ixz="0.0"
+                                   iyy="0.00144035" iyz="-0.00001139"
+                                                    izz="0.00198196"
         />
     </inertial>

File: xacro/leg.xacro (robot description, xacro)
@@ -5,10 +5,10 @@
   <xacro:property name="base_2_HAA_x" value="${0.0 * 0.001}" />
   <xacro:property name="base_2_HAA_y" value="${63.6 * 0.001}" />
-  <xacro:property name="HAA_2_HFE_y" value="${14.0 * 0.001}" />
+  <xacro:property name="HAA_2_HFE_y" value="${14.5 * 0.001}" />
   <xacro:property name="HAA_2_HFE_z" value="${38.60 * 0.001}" />
   <xacro:property name="base_2_HFE_x" value="${0.00 * 0.001}" />
   <xacro:property name="base_2_HFE_y" value="${78.10 * 0.001}" />
   <xacro:property name="base_2_HFE_z" value="${38.60 * 0.001}" />
-  <xacro:property name="HFE_2_KFE_y" value="${37.45 * 0.001}" />
+  <xacro:property name="HFE_2_KFE_y" value="${37.4 * 0.001}" />
   <xacro:property name="HFE_2_KFE_z" value="${160.00 * 0.001}" />
   <xacro:property name="KFE_2_FOOT_y" value="${8.0 * 0.001}" />
@@ -38,18 +38,19 @@
         <!-- create a dummy shoulder link to join the two joints -->
         <inertial>
-          <mass value="0.14853845"/>
           <xacro:unless value="${is_right}">
             <!-- Left upper leg inertia -->
-            <origin xyz="-0.07870700 0.01 0." rpy="0 0 0" />
-            <inertia ixx="0.00003024" ixy="0.00004671" ixz="0.0"
-                                      iyy="0.00041193" iyz="0.0"
-                                                      izz="0.00041107"/>
+            <mass value="0.14004265"/>
+            <origin xyz="0.01708256 -0.00446892 -0.01095830" rpy="0 0 0" />
+            <inertia ixx="0.00007443" ixy="0.00000148" ixz="0.00002154"
+                                      iyy="0.00013847" iyz="-0.00001096"
+                                                       izz="0.00009002"/>
           </xacro:unless>
           <xacro:if value="${is_right}">
             <!-- Right upper leg inertia -->
-            <origin xyz="-0.07870700 -0.01 0." rpy="0 0 0" />
-            <inertia ixx="0.00003024" ixy="-0.00004671" ixz="0.0"
-                                      iyy="0.00041193" iyz="0.0"
-                                                      izz="0.00041107"/>
+            <mass value="0.14004412"/>
+            <origin xyz="0.01708233 0.00447099 -0.01095846" rpy="0 0 0" />
+            <inertia ixx="0.00007442" ixy="-0.00000148" ixz="0.00002154"
+                                      iyy="0.00013848"  iyz="0.00001095"
+                                                        izz="0.00009001"/>
           </xacro:if>
         </inertial>
@@ -131,9 +132,9 @@
         <!-- Left upper leg inertia -->
         <inertial>
-        <origin xyz="0.00001377 0.01935853 -0.07870700" rpy="0 0 0" />
-        <mass value="0.14853845"/>
-        <inertia ixx="0.00041107" ixy="0.0"         ixz="0.0"
-                                   iyy="0.00041193" iyz="0.00004671"
-                                                    izz="0.00003024"/>
+          <origin xyz="0.00001377 0.01935853 -0.07870700" rpy="0 0 0" />
+          <mass value="0.14853845"/>
+          <inertia ixx="0.00041107" ixy="0.00000000"  ixz="0.00000009"
+                                    iyy="0.00041193"  iyz="-0.00004671"
+                                                      izz="0.00003024"/>
         </inertial>
       </xacro:unless>
@@ -141,9 +142,9 @@
         <!-- Right upper leg inertia -->
         <inertial>
-        <origin xyz="-0.00001377 -0.01935853 -0.07870700" rpy="0 0 0" />
-        <mass value="0.14853845"/>
-        <inertia ixx="0.00041107" ixy="0.0"         ixz="0.0"
-                                   iyy="0.00041193" iyz="-0.00004671"
-                                                    izz="0.00003024"/>
+          <origin xyz="-0.00001377 -0.01935853 -0.07870700" rpy="0 0 0" />
+          <mass value="0.14853845"/>
+          <inertia ixx="0.00041107" ixy="0.00000000"  ixz="-0.00000009"
+                                    iyy="0.00041193"  iyz="0.00004671"
+                                                      izz="0.00003024"/>
         </inertial>
       </xacro:if>
@@ -160,5 +161,5 @@
         </geometry>
         <material name="${color_name}">
-            <color rgba="${color} ${opacity}"/>
+          <color rgba="${color} ${opacity}"/>
         </material>
       </visual>
@@ -175,5 +176,5 @@
         </geometry>
         <material name="${color_name}">
-            <color rgba="${color} ${opacity}"/>
+          <color rgba="${color} ${opacity}"/>
         </material>
       </collision>
@@ -206,9 +207,9 @@
         <!-- Left lower leg inertia -->
         <inertial>
-        <origin xyz="0.0 0.00787644 -0.08928215" rpy="0 0 0" />
-        <mass value="0.03070001"/>
-        <inertia ixx="0.00012024" ixy="0.0"         ixz="0.0"
-                                   iyy="0.00012029" iyz="0.00000305"
-                                                    izz="0.00000216"/>
+          <origin xyz="0.0 0.00836718 -0.09591877" rpy="0 0 0" />
+          <mass value="0.03117243"/>
+          <inertia ixx="0.00011487" ixy="0.00000000"  ixz="0.00000000"
+                                    iyy="0.00011556"  iyz="-0.00000190"
+                                                      izz="0.00000220"/>
         </inertial>
       </xacro:unless>
@@ -216,9 +217,9 @@
         <!-- Right lower leg inertia -->
         <inertial>
-        <origin xyz="0.0 0.00787644 -0.08928215" rpy="0 0 0" />
-        <mass value="0.03070001"/>
-        <inertia ixx="0.00012024" ixy="0.0"         ixz="0.0"
-                                   iyy="0.00012029" iyz="-0.00000305"
-                                                    izz="0.00000216"/>
+          <origin xyz="0.0 -0.00836718 -0.09591877" rpy="0 0 0" />
+          <mass value="0.03117243"/>
+          <inertia ixx="0.00011487" ixy="0.00000000"  ixz="0.00000000"
+                                    iyy="0.00011556"  iyz="0.00000190"
+                                                      izz="0.00000220"/>
         </inertial>
       </xacro:if>
@@ -235,5 +236,5 @@
         </geometry>
         <material name="${color_name}">
-            <color rgba="${color} ${opacity}"/>
+          <color rgba="${color} ${opacity}"/>
         </material>
       </visual>
@@ -250,5 +251,5 @@
         </geometry>
         <material name="${color_name}">
-            <color rgba="${color} ${opacity}"/>
+          <color rgba="${color} ${opacity}"/>
         </material>
       </collision>
@@ -280,9 +281,9 @@
       <inertial>
         <origin xyz="0 0 0.00035767" rpy="0 0 0" />
-        <mass value="0.00693606"/>
+        <mass value="0.00000000"/>
         <inertia ixx="0.00000057" ixy="0.0"         ixz="0.0"
-                                   iyy="0.00000084" iyz="0.0"
-                                                    izz="0.00000053"/>
-     </inertial>
+                 iyy="0.00000084" iyz="0.0"
+                 izz="0.00000053"/>
+      </inertial>
       <!-- FOOT VISUAL -->
       <visual>
@@ -292,5 +293,5 @@
         </geometry>
         <material name="${color_name}">
-            <color rgba="${color} ${opacity}"/>
+          <color rgba="${color} ${opacity}"/>
         </material>
       </visual>
@@ -299,8 +300,8 @@
         <origin xyz="0 0 0" rpy="0 0 0" />
         <geometry>
-            <mesh filename="package://robot_properties_bolt/meshes/${mesh_ext}/bolt_foot.${mesh_ext}"/>
-        </geometry>
-        <material name="${color_name}">
-            <color rgba="${color} ${opacity}"/>
+          <mesh filename="package://robot_properties_bolt/meshes/${mesh_ext}/bolt_foot.${mesh_ext}"/>
+        </geometry>
+        <material name="${color_name}">
+          <color rgba="${color} ${opacity}"/>
         </material>
       </collision>
