Commit message: Add new legs

File: xacro/bolt.urdf.xacro (robot description, xacro)
@@ -9,18 +9,15 @@
   <xacro:property name="opacity" value="1.0" />
   <xacro:property name="mesh_ext" value="stl" />
+  <xacro:property name="new_leg" value="true" />
   <!-- This file is based on: https://atlas.is.localnet/confluence/display/AMDW/Quadruped+URDF+Files -->
   <link name="base_link">
     <!-- BASE LINK INERTIAL -->
     <inertial>
-        <origin xyz="-0.00245656 -0.00078880 0.03308090" rpy="0 0 0" />
+        <origin xyz="0 0 0" rpy="0 0 0" />
         <mass value="0.61436936"/>
         <!-- The base is extremely symmetrical. -->
-        <!--inertia ixx="0.00578574" ixy="0.0" ixz="0.0"
-                 iyy="0.01938108" iyz="0.0"
-                 izz="0.02476124"
-        /-->
-        <inertia ixx="0.00132170" ixy="0.00000117" ixz="0.0"
-                                   iyy="0.00144035" iyz="-0.00001139"
-                                                    izz="0.00198196"
+        <inertia ixx="0.00578574" ixy="0.0" ixz="0.0"
+                                  iyy="0.01938108" iyz="0.0"
+                                                   izz="0.02476124"
         />
     </inertial>
@@ -62,5 +59,6 @@
       color_name="${color_name}"
       color="${color}"
-      opacity="${opacity}"/>
+      opacity="${opacity}"
+      new_leg="${new_leg}"/>
   <!-- Include the front right leg -->
   <xacro:leg
@@ -72,4 +70,5 @@
       color_name="${color_name}"
       color="${color}"
-      opacity="${opacity}"/>
+      opacity="${opacity}"
+      new_leg="${new_leg}"/>
 </robot>

File: xacro/leg.xacro (robot description, xacro)
@@ -5,157 +5,68 @@
   <xacro:property name="base_2_HAA_x" value="${0.0 * 0.001}" />
   <xacro:property name="base_2_HAA_y" value="${63.6 * 0.001}" />
+  <!--xacro:property name="base_2_HAA_x" value="${2.45656 * 0.001}" />
+  <xacro:property name="base_2_HAA_y" value="${63.6 * 0.001}" />
+  <xacro:property name="base_2_HAA_z" value="${33.0809 * 0.001}" /-->
   <xacro:property name="HAA_2_HFE_y" value="${14.5 * 0.001}" />
   <xacro:property name="HAA_2_HFE_z" value="${38.60 * 0.001}" />
-  <xacro:property name="base_2_HFE_x" value="${0.00 * 0.001}" />
-  <xacro:property name="base_2_HFE_y" value="${78.10 * 0.001}" />
-  <xacro:property name="base_2_HFE_z" value="${38.60 * 0.001}" />
   <xacro:property name="HFE_2_KFE_y" value="${37.4 * 0.001}" />
-  <xacro:property name="HFE_2_KFE_z" value="${160.00 * 0.001}" />
+  <xacro:property name="HFE_2_KFE_z" value="${200.00 * 0.001}" />
   <xacro:property name="KFE_2_FOOT_y" value="${8.0 * 0.001}" />
-  <xacro:property name="KFE_2_FOOT_z" value="${160.00 * 0.001}" />
+  <xacro:property name="KFE_2_FOOT_z" value="${200.00 * 0.001}" />
   <!-- Macro defining bolt leg. -->
   <xacro:macro name="leg" params="prefix is_front is_right has_side_motion
-                                  mesh_ext color_name color opacity">
-    <xacro:if value="${has_side_motion}">
-      <joint name="${prefix}_HAA" type="revolute">
-        <parent link="base_link"/>
-        <child link="${prefix}_SHOULDER"/>
-        <limit effort="1000" lower="-10" upper="10" velocity="1000"/>
-        <!-- joints rotates around the x-axis -->
-        <axis xyz="1 0 0"/>
-        <!-- placement of the joint -->
+                                  mesh_ext color_name color opacity new_leg">
+    <joint name="${prefix}_HAA" type="revolute">
+      <parent link="base_link"/>
+      <child link="${prefix}_SHOULDER"/>
+      <limit effort="1000" lower="-10" upper="10" velocity="1000"/>
+      <!-- joints rotates around the x-axis -->
+      <axis xyz="1 0 0"/>
+      <!-- placement of the joint -->
+      <xacro:unless value="${is_right}">
+        <origin xyz="${base_2_HAA_x} ${base_2_HAA_y} 0" rpy="0 0 0" />
+      </xacro:unless>
+      <xacro:if value="${is_right}">
+        <origin xyz="${base_2_HAA_x} ${-base_2_HAA_y} 0" rpy="0 0 0" />
+      </xacro:if>
+      <!--xacro:unless value="${is_right}">
+        <origin xyz="${base_2_HAA_x} ${base_2_HAA_y + 0.0007888} ${-base_2_HAA_z}" rpy="0 0 0" />
+      </xacro:unless>
+      <xacro:if value="${is_right}">
+        <origin xyz="${base_2_HAA_x} ${-base_2_HAA_y + 0.0007888} ${-base_2_HAA_z}" rpy="0 0 0" />
+      </xacro:if-->
+      <!-- pybullet simulation parameters -->
+      <dynamics damping="0.0" friction="0.0"/>
+    </joint>
+    <link name="${prefix}_SHOULDER">
+      <!-- TODO: Update inertias and add visuals for link. -->
+      <!-- create a dummy shoulder link to join the two joints -->
+      <inertial>
         <xacro:unless value="${is_right}">
-          <origin xyz="${base_2_HAA_x} ${base_2_HAA_y} 0" rpy="0 0 0" />
+          <!-- Left upper leg inertia -->
+          <mass value="0.14004265"/>
+          <origin xyz="0.01708256 -0.00446892 -0.01095830" rpy="0 0 0" />
+          <inertia ixx="0.00007443" ixy="0.00000148" ixz="0.00002154"
+                   iyy="0.00013847" iyz="-0.00001096"
+                   izz="0.00009002"/>
         </xacro:unless>
         <xacro:if value="${is_right}">
-          <origin xyz="${base_2_HAA_x} ${-base_2_HAA_y} 0" rpy="0 0 0" />
+          <!-- Right upper leg inertia -->
+          <mass value="0.14004412"/>
+          <origin xyz="0.01708233 0.00447099 -0.01095846" rpy="0 0 0" />
+          <inertia ixx="0.00007442" ixy="-0.00000148" ixz="0.00002154"
+                   iyy="0.00013848"  iyz="0.00001095"
+                   izz="0.00009001"/>
         </xacro:if>
-        <!-- pybullet simulation parameters -->
-        <dynamics damping="0.0" friction="0.0"/>
-      </joint>
-      <link name="${prefix}_SHOULDER">
-        <!-- TODO: Update inertias and add visuals for link. -->
-        <!-- create a dummy shoulder link to join the two joints -->
-        <inertial>
+      </inertial>
+      <!-- HIP LEG LINK VISUAL -->
+      <visual>
+        <origin xyz="0 0 0" rpy="0 0 0" />
+        <geometry>
           <xacro:unless value="${is_right}">
-            <!-- Left upper leg inertia -->
-            <mass value="0.14004265"/>
-            <origin xyz="0.01708256 -0.00446892 -0.01095830" rpy="0 0 0" />
-            <inertia ixx="0.00007443" ixy="0.00000148" ixz="0.00002154"
-                                      iyy="0.00013847" iyz="-0.00001096"
-                                                       izz="0.00009002"/>
+            <mesh filename="package://robot_properties_bolt/meshes/${mesh_ext}/bolt_hip_fe_left_side.${mesh_ext}"/>
           </xacro:unless>
           <xacro:if value="${is_right}">
-            <!-- Right upper leg inertia -->
-            <mass value="0.14004412"/>
-            <origin xyz="0.01708233 0.00447099 -0.01095846" rpy="0 0 0" />
-            <inertia ixx="0.00007442" ixy="-0.00000148" ixz="0.00002154"
-                                      iyy="0.00013848"  iyz="0.00001095"
-                                                        izz="0.00009001"/>
-          </xacro:if>
-        </inertial>
-        <!-- UPPER LEG LINK VISUAL -->
-        <visual>
-          <origin xyz="0 0 0" rpy="0 0 0" />
-          <geometry>
-            <xacro:unless value="${is_right}">
-              <mesh filename="package://robot_properties_bolt/meshes/${mesh_ext}/bolt_hip_fe_left_side.${mesh_ext}"/>
-            </xacro:unless>
-            <xacro:if value="${is_right}">
-              <mesh filename="package://robot_properties_bolt/meshes/${mesh_ext}/bolt_hip_fe_right_side.${mesh_ext}"/>
-            </xacro:if>
-          </geometry>
-          <material name="${color_name}">
-            <color rgba="${color} ${opacity}"/>
-          </material>
-        </visual>
-        <!-- UPPER LEG LINK COLLISION -->
-        <collision>
-          <origin xyz="0 0 0" rpy="0 0 0" />
-          <geometry>
-            <xacro:unless value="${is_right}">
-              <mesh filename="package://robot_properties_bolt/meshes/${mesh_ext}/bolt_upper_leg_left_side.${mesh_ext}"/>
-            </xacro:unless>
-            <xacro:if value="${is_right}">
-              <mesh filename="package://robot_properties_bolt/meshes/${mesh_ext}/bolt_upper_leg_right_side.${mesh_ext}"/>
-            </xacro:if>
-          </geometry>
-          <material name="${color_name}">
-            <color rgba="${color} ${opacity}"/>
-          </material>
-        </collision>
-        <!-- Bullet specific paramters -->
-        <contact>
-          <lateral_friction value="1.0"/>
-          <restitution value="0.5"/>
-        </contact>
-      </link>
-      <joint name="${prefix}_HFE" type="revolute">
-        <parent link="${prefix}_SHOULDER"/>
-        <child link="${prefix}_UPPER_LEG"/>
-        <limit effort="1000" lower="-10" upper="10" velocity="1000"/>
-        <!-- joints rotates around the y-axis -->
-        <axis xyz="0 1 0"/>
-        <!-- placement of the joint -->
-        <xacro:if value="${is_right}">
-          <origin xyz="0 ${-HAA_2_HFE_y} ${-HAA_2_HFE_z}" rpy="0 0 0" />
-        </xacro:if>
-        <xacro:unless value="${is_right}">
-          <origin xyz="0 ${HAA_2_HFE_y} ${-HAA_2_HFE_z}" rpy="0 0 0" />
-        </xacro:unless>
-        <!-- pybullet simulation parameters -->
-        <dynamics damping="0.0" friction="0.0"/>
-      </joint>
-    </xacro:if>
-    <xacro:unless value="${has_side_motion}">
-      <!-- Joint between the base and the ${prefix} upper leg -->
-      <joint name="${prefix}_HFE" type="revolute">
-        <parent link="base_link"/>
-        <child link="${prefix}_UPPER_LEG"/>
-        <limit effort="1000" lower="-10" upper="10" velocity="1000"/>
-        <!-- joints rotates around the y-axis -->
-        <axis xyz="0 1 0"/>
-        <!-- placement of the joint -->
-        <xacro:unless value="${is_right}">
-          <origin xyz="${base_2_HFE_x} ${base_2_HFE_y} ${base_2_HFE_z}" rpy="0 0 0" />
-        </xacro:unless>
-        <xacro:if value="${is_right}">
-          <origin xyz="${base_2_HFE_x} ${-base_2_HFE_y} ${base_2_HFE_z}" rpy="0 0 0" />
-        </xacro:if>
-        <!-- pybullet simulation parameters -->
-        <dynamics damping="0.0" friction="0.0"/>
-      </joint>
-    </xacro:unless>
-    <link name="${prefix}_UPPER_LEG">
-      <!-- UPPER LEG LINK INERTIAL -->
-      <xacro:unless value="${is_right}">
-        <!-- Left upper leg inertia -->
-        <inertial>
-          <origin xyz="0.00001377 0.01935853 -0.07870700" rpy="0 0 0" />
-          <mass value="0.14853845"/>
-          <inertia ixx="0.00041107" ixy="0.00000000"  ixz="0.00000009"
-                                    iyy="0.00041193"  iyz="-0.00004671"
-                                                      izz="0.00003024"/>
-        </inertial>
-      </xacro:unless>
-      <xacro:if value="${is_right}">
-        <!-- Right upper leg inertia -->
-        <inertial>
-          <origin xyz="-0.00001377 -0.01935853 -0.07870700" rpy="0 0 0" />
-          <mass value="0.14853845"/>
-          <inertia ixx="0.00041107" ixy="0.00000000"  ixz="-0.00000009"
-                                    iyy="0.00041193"  iyz="0.00004671"
-                                                      izz="0.00003024"/>
-        </inertial>
-      </xacro:if>
-      <!-- UPPER LEG LINK VISUAL -->
-      <visual>
-        <origin xyz="0 0 0" rpy="0 0 0" />
-        <geometry>
-          <xacro:unless value="${is_right}">
-            <mesh filename="package://robot_properties_bolt/meshes/${mesh_ext}/bolt_upper_leg_left_side.${mesh_ext}"/>
-          </xacro:unless>
-          <xacro:if value="${is_right}">
-            <mesh filename="package://robot_properties_bolt/meshes/${mesh_ext}/bolt_upper_leg_right_side.${mesh_ext}"/>
+            <mesh filename="package://robot_properties_bolt/meshes/${mesh_ext}/bolt_hip_fe_right_side.${mesh_ext}"/>
           </xacro:if>
         </geometry>
@@ -169,8 +80,102 @@
         <geometry>
           <xacro:unless value="${is_right}">
-            <mesh filename="package://robot_properties_bolt/meshes/${mesh_ext}/bolt_upper_leg_left_side.${mesh_ext}"/>
+            <mesh filename="package://robot_properties_bolt/meshes/${mesh_ext}/bolt_hip_fe_left_side.${mesh_ext}"/>
           </xacro:unless>
           <xacro:if value="${is_right}">
-            <mesh filename="package://robot_properties_bolt/meshes/${mesh_ext}/bolt_upper_leg_right_side.${mesh_ext}"/>
+            <mesh filename="package://robot_properties_bolt/meshes/${mesh_ext}/bolt_hip_fe_right_side.${mesh_ext}"/>
+          </xacro:if>
+        </geometry>
+        <material name="${color_name}">
+          <color rgba="${color} ${opacity}"/>
+        </material>
+      </collision>
+      <!-- Bullet specific paramters -->
+      <contact>
+        <lateral_friction value="1.0"/>
+        <restitution value="0.5"/>
+      </contact>
+    </link>
+    <joint name="${prefix}_HFE" type="revolute">
+      <parent link="${prefix}_SHOULDER"/>
+      <child link="${prefix}_UPPER_LEG"/>
+      <limit effort="1000" lower="-10" upper="10" velocity="1000"/>
+      <!-- joints rotates around the y-axis -->
+      <axis xyz="0 1 0"/>
+      <!-- placement of the joint -->
+      <xacro:if value="${is_right}">
+        <origin xyz="0 ${-HAA_2_HFE_y} ${-HAA_2_HFE_z}" rpy="0 0 0" />
+      </xacro:if>
+      <xacro:unless value="${is_right}">
+        <origin xyz="0 ${HAA_2_HFE_y} ${-HAA_2_HFE_z}" rpy="0 0 0" />
+      </xacro:unless>
+      <!-- pybullet simulation parameters -->
+      <dynamics damping="0.0" friction="0.0"/>
+    </joint>
+    <link name="${prefix}_UPPER_LEG">
+      <!-- UPPER LEG LINK INERTIAL -->
+      <xacro:unless value="${is_right}">
+        <!-- Left upper leg inertia -->
+        <inertial>
+          <origin xyz="0.00001377 0.01935853 -0.11870700" rpy="0 0 0" />
+          <mass value="0.14853845"/>
+          <inertia ixx="0.00041107" ixy="0.00000000"  ixz="0.00000009"
+                   iyy="0.00041193"  iyz="-0.00004671"
+                   izz="0.00003024"/>
+        </inertial>
+      </xacro:unless>
+      <xacro:if value="${is_right}">
+        <!-- Right upper leg inertia -->
+        <inertial>
+          <origin xyz="-0.00001377 -0.01935853 -0.11870700" rpy="0 0 0" />
+          <mass value="0.14853845"/>
+          <inertia ixx="0.00041107" ixy="0.00000000"  ixz="-0.00000009"
+                   iyy="0.00041193"  iyz="0.00004671"
+                   izz="0.00003024"/>
+        </inertial>
+      </xacro:if>
+      <!-- UPPER LEG LINK VISUAL -->
+      <visual>
+        <origin xyz="0 0 0" rpy="0 0 0" />
+        <geometry>
+          <xacro:unless value="${new_leg}">
+            <xacro:unless value="${is_right}">
+              <mesh filename="package://robot_properties_bolt/meshes/${mesh_ext}/bolt_upper_leg_left_side.${mesh_ext}"/>
+            </xacro:unless>
+            <xacro:if value="${is_right}">
+              <mesh filename="package://robot_properties_bolt/meshes/${mesh_ext}/bolt_upper_leg_right_side.${mesh_ext}"/>
+            </xacro:if>
+          </xacro:unless>
+          <xacro:if value="${new_leg}">
+            <xacro:unless value="${is_right}">
+              <mesh filename="package://robot_properties_bolt/meshes/${mesh_ext}/upper_leg_200mm_left_side.${mesh_ext}"/>
+            </xacro:unless>
+            <xacro:if value="${is_right}">
+              <mesh filename="package://robot_properties_bolt/meshes/${mesh_ext}/upper_leg_200mm_right_side.${mesh_ext}"/>
+            </xacro:if>
+          </xacro:if>
+        </geometry>
+        <material name="${color_name}">
+          <color rgba="${color} ${opacity}"/>
+        </material>
+      </visual>
+      <!-- UPPER LEG LINK COLLISION -->
+      <collision>
+        <origin xyz="0 0 0" rpy="0 0 0" />
+        <geometry>
+          <xacro:unless value="${new_leg}">
+            <xacro:unless value="${is_right}">
+              <mesh filename="package://robot_properties_bolt/meshes/${mesh_ext}/bolt_upper_leg_left_side.${mesh_ext}"/>
+            </xacro:unless>
+            <xacro:if value="${is_right}">
+              <mesh filename="package://robot_properties_bolt/meshes/${mesh_ext}/bolt_upper_leg_right_side.${mesh_ext}"/>
+            </xacro:if>
+          </xacro:unless>
+          <xacro:if value="${new_leg}">
+            <xacro:unless value="${is_right}">
+              <mesh filename="package://robot_properties_bolt/meshes/${mesh_ext}/upper_leg_200mm_left_side.${mesh_ext}"/>
+            </xacro:unless>
+            <xacro:if value="${is_right}">
+              <mesh filename="package://robot_properties_bolt/meshes/${mesh_ext}/upper_leg_200mm_right_side.${mesh_ext}"/>
+            </xacro:if>
           </xacro:if>
         </geometry>
@@ -207,9 +212,9 @@
         <!-- Left lower leg inertia -->
         <inertial>
-          <origin xyz="0.0 0.00836718 -0.09591877" rpy="0 0 0" />
+          <origin xyz="0.0 0.00836718 -0.11591877" rpy="0 0 0" />
           <mass value="0.03117243"/>
           <inertia ixx="0.00011487" ixy="0.00000000"  ixz="0.00000000"
-                                    iyy="0.00011556"  iyz="-0.00000190"
-                                                      izz="0.00000220"/>
+                   iyy="0.00011556"  iyz="-0.00000190"
+                   izz="0.00000220"/>
         </inertial>
       </xacro:unless>
@@ -217,9 +222,9 @@
         <!-- Right lower leg inertia -->
         <inertial>
-          <origin xyz="0.0 -0.00836718 -0.09591877" rpy="0 0 0" />
+          <origin xyz="0.0 -0.00836718 -0.11591877" rpy="0 0 0" />
           <mass value="0.03117243"/>
           <inertia ixx="0.00011487" ixy="0.00000000"  ixz="0.00000000"
-                                    iyy="0.00011556"  iyz="0.00000190"
-                                                      izz="0.00000220"/>
+                   iyy="0.00011556"  iyz="0.00000190"
+                   izz="0.00000220"/>
         </inertial>
       </xacro:if>
@@ -228,9 +233,19 @@
         <origin xyz="0 0 0" rpy="0 0 0" />
         <geometry>
-          <xacro:unless value="${is_right}">
-            <mesh filename="package://robot_properties_bolt/meshes/${mesh_ext}/bolt_lower_leg_left_side.${mesh_ext}"/>
-          </xacro:unless>
-          <xacro:if value="${is_right}">
-            <mesh filename="package://robot_properties_bolt/meshes/${mesh_ext}/bolt_lower_leg_right_side.${mesh_ext}"/>
+          <xacro:unless value="${new_leg}">
+            <xacro:unless value="${is_right}">
+              <mesh filename="package://robot_properties_bolt/meshes/${mesh_ext}/bolt_lower_leg_left_side.${mesh_ext}"/>
+            </xacro:unless>
+            <xacro:if value="${is_right}">
+              <mesh filename="package://robot_properties_bolt/meshes/${mesh_ext}/bolt_lower_leg_right_side.${mesh_ext}"/>
+            </xacro:if>
+          </xacro:unless>
+          <xacro:if value="${new_leg}">
+            <xacro:unless value="${is_right}">
+              <mesh filename="package://robot_properties_bolt/meshes/${mesh_ext}/lower_leg_200mm_left_side.${mesh_ext}"/>
+            </xacro:unless>
+            <xacro:if value="${is_right}">
+              <mesh filename="package://robot_properties_bolt/meshes/${mesh_ext}/lower_leg_200mm_right_side.${mesh_ext}"/>
+            </xacro:if>
           </xacro:if>
         </geometry>
@@ -243,9 +258,19 @@
         <origin xyz="0 0 0" rpy="0 0 0" />
         <geometry>
-          <xacro:unless value="${is_right}">
-            <mesh filename="package://robot_properties_bolt/meshes/${mesh_ext}/bolt_lower_leg_left_side.${mesh_ext}"/>
-          </xacro:unless>
-          <xacro:if value="${is_right}">
-            <mesh filename="package://robot_properties_bolt/meshes/${mesh_ext}/bolt_lower_leg_right_side.${mesh_ext}"/>
+          <xacro:unless value="${new_leg}">
+            <xacro:unless value="${is_right}">
+              <mesh filename="package://robot_properties_bolt/meshes/${mesh_ext}/bolt_lower_leg_left_side.${mesh_ext}"/>
+            </xacro:unless>
+            <xacro:if value="${is_right}">
+              <mesh filename="package://robot_properties_bolt/meshes/${mesh_ext}/bolt_lower_leg_right_side.${mesh_ext}"/>
+            </xacro:if>
+          </xacro:unless>
+          <xacro:if value="${new_leg}">
+            <xacro:unless value="${is_right}">
+              <mesh filename="package://robot_properties_bolt/meshes/${mesh_ext}/lower_leg_200mm_left_side.${mesh_ext}"/>
+            </xacro:unless>
+            <xacro:if value="${is_right}">
+              <mesh filename="package://robot_properties_bolt/meshes/${mesh_ext}/lower_leg_200mm_right_side.${mesh_ext}"/>
+            </xacro:if>
           </xacro:if>
         </geometry>
