Commit message: made repo pip installable

File: src/robot_properties_bolt/resources/pre_generated_urdf/bolt.urdf (robot description, URDF)
Before this commit: robot bolt, 9 links, 8 joints
Links:
- link FL_FOOT: geometry collision mesh filename=package://meshes/stl/bolt_foot.stl; visual mesh filename=package://meshes/stl/bolt_foot.stl
- link FL_LOWER_LEG: geometry collision mesh filename=package://meshes/stl/lower_leg_200mm_left_side.stl; visual mesh filename=package://meshes/stl/lower_leg_200mm_left_side.stl
- link FL_SHOULDER: geometry collision mesh filename=package://meshes/stl/bolt_hip_fe_left_side.stl; visual mesh filename=package://meshes/stl/bolt_hip_fe_left_side.stl
- link FL_UPPER_LEG: geometry collision mesh filename=package://meshes/stl/upper_leg_200mm_left_side.stl; visual mesh filename=package://meshes/stl/upper_leg_200mm_left_side.stl
- link FR_FOOT: geometry collision mesh filename=package://meshes/stl/bolt_foot.stl; visual mesh filename=package://meshes/stl/bolt_foot.stl
- link FR_LOWER_LEG: geometry collision mesh filename=package://meshes/stl/lower_leg_200mm_right_side.stl; visual mesh filename=package://meshes/stl/lower_leg_200mm_right_side.stl
- link FR_SHOULDER: geometry collision mesh filename=package://meshes/stl/bolt_hip_fe_right_side.stl; visual mesh filename=package://meshes/stl/bolt_hip_fe_right_side.stl
- link FR_UPPER_LEG: geometry collision mesh filename=package://meshes/stl/upper_leg_200mm_right_side.stl; visual mesh filename=package://meshes/stl/upper_leg_200mm_right_side.stl
- link base_link: geometry collision mesh filename=package://meshes/stl/bolt_body.stl; visual mesh filename=package://meshes/stl/bolt_body.stl
Joints:
- joint FL_ANKLE: origin xyz=0 0.008 -0.16 rpy=0 0 0 -> xyz=0 0.008 -0.2 rpy=0 0 0
- joint FL_KFE: origin xyz=0 0.0374 -0.16 rpy=0 0 0 -> xyz=0 0.0374 -0.2 rpy=0 0 0
- joint FR_ANKLE: origin xyz=0 -0.008 -0.16 rpy=0 0 0 -> xyz=0 -0.008 -0.2 rpy=0 0 0
- joint FR_KFE: origin xyz=0 -0.0374 -0.16 rpy=0 0 0 -> xyz=0 -0.0374 -0.2 rpy=0 0 0

File: src/robot_properties_bolt/resources/pre_generated_urdf/plane_with_restitution.urdf (robot description, URDF)
Before this commit: robot plane, 1 links, 0 joints
Links:
- link planeLink: geometry collision box size=30 30 10; visual mesh filename=package://meshes/plane.obj scale=1 1 1

File: src/robot_properties_bolt/resources/xacro/bolt.urdf.xacro (robot description, xacro)
@@ -26,5 +26,5 @@
         <origin xyz="0 0 0" rpy="0 0 0" />
         <geometry>
-          <mesh filename="package://robot_properties_bolt/meshes/${mesh_ext}/bolt_body.${mesh_ext}"/>
+          <mesh filename="package://meshes/${mesh_ext}/bolt_body.${mesh_ext}"/>
         </geometry>
         <material name="${color_name}">
@@ -36,5 +36,5 @@
         <origin xyz="0 0 0" rpy="0 0 0" />
         <geometry>
-          <mesh filename="package://robot_properties_bolt/meshes/${mesh_ext}/bolt_body.${mesh_ext}"/>
+          <mesh filename="package://meshes/${mesh_ext}/bolt_body.${mesh_ext}"/>
         </geometry>
         <material name="${color_name}">

File: src/robot_properties_bolt/resources/xacro/leg.xacro (robot description, xacro)
@@ -65,8 +65,8 @@
         <geometry>
           <xacro:unless value="${is_right}">
-            <mesh filename="package://robot_properties_bolt/meshes/${mesh_ext}/bolt_hip_fe_left_side.${mesh_ext}"/>
+            <mesh filename="package://meshes/${mesh_ext}/bolt_hip_fe_left_side.${mesh_ext}"/>
           </xacro:unless>
           <xacro:if value="${is_right}">
-            <mesh filename="package://robot_properties_bolt/meshes/${mesh_ext}/bolt_hip_fe_right_side.${mesh_ext}"/>
+            <mesh filename="package://meshes/${mesh_ext}/bolt_hip_fe_right_side.${mesh_ext}"/>
           </xacro:if>
         </geometry>
@@ -80,8 +80,8 @@
         <geometry>
           <xacro:unless value="${is_right}">
-            <mesh filename="package://robot_properties_bolt/meshes/${mesh_ext}/bolt_hip_fe_left_side.${mesh_ext}"/>
+            <mesh filename="package://meshes/${mesh_ext}/bolt_hip_fe_left_side.${mesh_ext}"/>
           </xacro:unless>
           <xacro:if value="${is_right}">
-            <mesh filename="package://robot_properties_bolt/meshes/${mesh_ext}/bolt_hip_fe_right_side.${mesh_ext}"/>
+            <mesh filename="package://meshes/${mesh_ext}/bolt_hip_fe_right_side.${mesh_ext}"/>
           </xacro:if>
         </geometry>
@@ -140,16 +140,16 @@
           <xacro:unless value="${new_leg}">
             <xacro:unless value="${is_right}">
-              <mesh filename="package://robot_properties_bolt/meshes/${mesh_ext}/bolt_upper_leg_left_side.${mesh_ext}"/>
-            </xacro:unless>
-            <xacro:if value="${is_right}">
-              <mesh filename="package://robot_properties_bolt/meshes/${mesh_ext}/bolt_upper_leg_right_side.${mesh_ext}"/>
+              <mesh filename="package://meshes/${mesh_ext}/bolt_upper_leg_left_side.${mesh_ext}"/>
+            </xacro:unless>
+            <xacro:if value="${is_right}">
+              <mesh filename="package://meshes/${mesh_ext}/bolt_upper_leg_right_side.${mesh_ext}"/>
             </xacro:if>
           </xacro:unless>
           <xacro:if value="${new_leg}">
             <xacro:unless value="${is_right}">
-              <mesh filename="package://robot_properties_bolt/meshes/${mesh_ext}/upper_leg_200mm_left_side.${mesh_ext}"/>
-            </xacro:unless>
-            <xacro:if value="${is_right}">
-              <mesh filename="package://robot_properties_bolt/meshes/${mesh_ext}/upper_leg_200mm_right_side.${mesh_ext}"/>
+              <mesh filename="package://meshes/${mesh_ext}/upper_leg_200mm_left_side.${mesh_ext}"/>
+            </xacro:unless>
+            <xacro:if value="${is_right}">
+              <mesh filename="package://meshes/${mesh_ext}/upper_leg_200mm_right_side.${mesh_ext}"/>
             </xacro:if>
           </xacro:if>
@@ -165,16 +165,16 @@
           <xacro:unless value="${new_leg}">
             <xacro:unless value="${is_right}">
-              <mesh filename="package://robot_properties_bolt/meshes/${mesh_ext}/bolt_upper_leg_left_side.${mesh_ext}"/>
-            </xacro:unless>
-            <xacro:if value="${is_right}">
-              <mesh filename="package://robot_properties_bolt/meshes/${mesh_ext}/bolt_upper_leg_right_side.${mesh_ext}"/>
+              <mesh filename="package://meshes/${mesh_ext}/bolt_upper_leg_left_side.${mesh_ext}"/>
+            </xacro:unless>
+            <xacro:if value="${is_right}">
+              <mesh filename="package://meshes/${mesh_ext}/bolt_upper_leg_right_side.${mesh_ext}"/>
             </xacro:if>
           </xacro:unless>
           <xacro:if value="${new_leg}">
             <xacro:unless value="${is_right}">
-              <mesh filename="package://robot_properties_bolt/meshes/${mesh_ext}/upper_leg_200mm_left_side.${mesh_ext}"/>
-            </xacro:unless>
-            <xacro:if value="${is_right}">
-              <mesh filename="package://robot_properties_bolt/meshes/${mesh_ext}/upper_leg_200mm_right_side.${mesh_ext}"/>
+              <mesh filename="package://meshes/${mesh_ext}/upper_leg_200mm_left_side.${mesh_ext}"/>
+            </xacro:unless>
+            <xacro:if value="${is_right}">
+              <mesh filename="package://meshes/${mesh_ext}/upper_leg_200mm_right_side.${mesh_ext}"/>
             </xacro:if>
           </xacro:if>
@@ -235,16 +235,16 @@
           <xacro:unless value="${new_leg}">
             <xacro:unless value="${is_right}">
-              <mesh filename="package://robot_properties_bolt/meshes/${mesh_ext}/bolt_lower_leg_left_side.${mesh_ext}"/>
-            </xacro:unless>
-            <xacro:if value="${is_right}">
-              <mesh filename="package://robot_properties_bolt/meshes/${mesh_ext}/bolt_lower_leg_right_side.${mesh_ext}"/>
+              <mesh filename="package://meshes/${mesh_ext}/bolt_lower_leg_left_side.${mesh_ext}"/>
+            </xacro:unless>
+            <xacro:if value="${is_right}">
+              <mesh filename="package://meshes/${mesh_ext}/bolt_lower_leg_right_side.${mesh_ext}"/>
             </xacro:if>
           </xacro:unless>
           <xacro:if value="${new_leg}">
             <xacro:unless value="${is_right}">
-              <mesh filename="package://robot_properties_bolt/meshes/${mesh_ext}/lower_leg_200mm_left_side.${mesh_ext}"/>
-            </xacro:unless>
-            <xacro:if value="${is_right}">
-              <mesh filename="package://robot_properties_bolt/meshes/${mesh_ext}/lower_leg_200mm_right_side.${mesh_ext}"/>
+              <mesh filename="package://meshes/${mesh_ext}/lower_leg_200mm_left_side.${mesh_ext}"/>
+            </xacro:unless>
+            <xacro:if value="${is_right}">
+              <mesh filename="package://meshes/${mesh_ext}/lower_leg_200mm_right_side.${mesh_ext}"/>
             </xacro:if>
           </xacro:if>
@@ -260,16 +260,16 @@
           <xacro:unless value="${new_leg}">
             <xacro:unless value="${is_right}">
-              <mesh filename="package://robot_properties_bolt/meshes/${mesh_ext}/bolt_lower_leg_left_side.${mesh_ext}"/>
-            </xacro:unless>
-            <xacro:if value="${is_right}">
-              <mesh filename="package://robot_properties_bolt/meshes/${mesh_ext}/bolt_lower_leg_right_side.${mesh_ext}"/>
+              <mesh filename="package://meshes/${mesh_ext}/bolt_lower_leg_left_side.${mesh_ext}"/>
+            </xacro:unless>
+            <xacro:if value="${is_right}">
+              <mesh filename="package://meshes/${mesh_ext}/bolt_lower_leg_right_side.${mesh_ext}"/>
             </xacro:if>
           </xacro:unless>
           <xacro:if value="${new_leg}">
             <xacro:unless value="${is_right}">
-              <mesh filename="package://robot_properties_bolt/meshes/${mesh_ext}/lower_leg_200mm_left_side.${mesh_ext}"/>
-            </xacro:unless>
-            <xacro:if value="${is_right}">
-              <mesh filename="package://robot_properties_bolt/meshes/${mesh_ext}/lower_leg_200mm_right_side.${mesh_ext}"/>
+              <mesh filename="package://meshes/${mesh_ext}/lower_leg_200mm_left_side.${mesh_ext}"/>
+            </xacro:unless>
+            <xacro:if value="${is_right}">
+              <mesh filename="package://meshes/${mesh_ext}/lower_leg_200mm_right_side.${mesh_ext}"/>
             </xacro:if>
           </xacro:if>
@@ -315,5 +315,5 @@
         <origin xyz="0 0 0" rpy="0 0 0" />
         <geometry>
-          <mesh filename="package://robot_properties_bolt/meshes/${mesh_ext}/bolt_foot.${mesh_ext}"/>
+          <mesh filename="package://meshes/${mesh_ext}/bolt_foot.${mesh_ext}"/>
         </geometry>
         <material name="${color_name}">
@@ -325,5 +325,5 @@
         <origin xyz="0 0 0" rpy="0 0 0" />
         <geometry>
-          <mesh filename="package://robot_properties_bolt/meshes/${mesh_ext}/bolt_foot.${mesh_ext}"/>
+          <mesh filename="package://meshes/${mesh_ext}/bolt_foot.${mesh_ext}"/>
         </geometry>
         <material name="${color_name}">

File: src/robot_properties_bolt/resources/xacro/plane_with_restitution.urdf.xacro (robot description, xacro)
@@ -15,5 +15,5 @@
       <origin rpy="0 0 0" xyz="0 0 0"/>
       <geometry>
-      <mesh filename="package://robot_properties_bolt/meshes/plane.obj" scale="1 1 1"/>
+      <mesh filename="package://meshes/plane.obj" scale="1 1 1"/>
       </geometry>
        <material name="white">
