Commit message: included package name in the mesh path in xacro files; changed yaml_path to dgm_yaml_path; removed xacro encoding for python2

File: src/robot_properties_bolt/robot_properties_bolt/xacro/bolt.urdf.xacro (robot description, xacro)
@@ -26,5 +26,5 @@
         <origin xyz="0 0 0" rpy="0 0 0" />
         <geometry>
-          <mesh filename="package://meshes/${mesh_ext}/bolt_body.${mesh_ext}"/>
+          <mesh filename="package://robot_properties_bolt/meshes/${mesh_ext}/bolt_body.${mesh_ext}"/>
         </geometry>
         <material name="${color_name}">
@@ -36,5 +36,5 @@
         <origin xyz="0 0 0" rpy="0 0 0" />
         <geometry>
-          <mesh filename="package://meshes/${mesh_ext}/bolt_body.${mesh_ext}"/>
+          <mesh filename="package://robot_properties_bolt/meshes/${mesh_ext}/bolt_body.${mesh_ext}"/>
         </geometry>
         <material name="${color_name}">

File: src/robot_properties_bolt/robot_properties_bolt/xacro/leg.xacro (robot description, xacro)
@@ -65,8 +65,8 @@
         <geometry>
           <xacro:unless value="${is_right}">
-            <mesh filename="package://meshes/${mesh_ext}/bolt_hip_fe_left_side.${mesh_ext}"/>
+            <mesh filename="package://robot_properties_bolt/meshes/${mesh_ext}/bolt_hip_fe_left_side.${mesh_ext}"/>
           </xacro:unless>
           <xacro:if value="${is_right}">
-            <mesh filename="package://meshes/${mesh_ext}/bolt_hip_fe_right_side.${mesh_ext}"/>
+            <mesh filename="package://robot_properties_bolt/meshes/${mesh_ext}/bolt_hip_fe_right_side.${mesh_ext}"/>
           </xacro:if>
         </geometry>
@@ -80,8 +80,8 @@
         <geometry>
           <xacro:unless value="${is_right}">
-            <mesh filename="package://meshes/${mesh_ext}/bolt_hip_fe_left_side.${mesh_ext}"/>
+            <mesh filename="package://robot_properties_bolt/meshes/${mesh_ext}/bolt_hip_fe_left_side.${mesh_ext}"/>
           </xacro:unless>
           <xacro:if value="${is_right}">
-            <mesh filename="package://meshes/${mesh_ext}/bolt_hip_fe_right_side.${mesh_ext}"/>
+            <mesh filename="package://robot_properties_bolt/meshes/${mesh_ext}/bolt_hip_fe_right_side.${mesh_ext}"/>
           </xacro:if>
         </geometry>
@@ -140,16 +140,16 @@
           <xacro:unless value="${new_leg}">
             <xacro:unless value="${is_right}">
-              <mesh filename="package://meshes/${mesh_ext}/bolt_upper_leg_left_side.${mesh_ext}"/>
-            </xacro:unless>
-            <xacro:if value="${is_right}">
-              <mesh filename="package://meshes/${mesh_ext}/bolt_upper_leg_right_side.${mesh_ext}"/>
+              <mesh filename="package://robot_properties_bolt/meshes/${mesh_ext}/bolt_upper_leg_left_side.${mesh_ext}"/>
+            </xacro:unless>
+            <xacro:if value="${is_right}">
+              <mesh filename="package://robot_properties_bolt/meshes/${mesh_ext}/bolt_upper_leg_right_side.${mesh_ext}"/>
             </xacro:if>
           </xacro:unless>
           <xacro:if value="${new_leg}">
             <xacro:unless value="${is_right}">
-              <mesh filename="package://meshes/${mesh_ext}/upper_leg_200mm_left_side.${mesh_ext}"/>
-            </xacro:unless>
-            <xacro:if value="${is_right}">
-              <mesh filename="package://meshes/${mesh_ext}/upper_leg_200mm_right_side.${mesh_ext}"/>
+              <mesh filename="package://robot_properties_bolt/meshes/${mesh_ext}/upper_leg_200mm_left_side.${mesh_ext}"/>
+            </xacro:unless>
+            <xacro:if value="${is_right}">
+              <mesh filename="package://robot_properties_bolt/meshes/${mesh_ext}/upper_leg_200mm_right_side.${mesh_ext}"/>
             </xacro:if>
           </xacro:if>
@@ -165,16 +165,16 @@
           <xacro:unless value="${new_leg}">
             <xacro:unless value="${is_right}">
-              <mesh filename="package://meshes/${mesh_ext}/bolt_upper_leg_left_side.${mesh_ext}"/>
-            </xacro:unless>
-            <xacro:if value="${is_right}">
-              <mesh filename="package://meshes/${mesh_ext}/bolt_upper_leg_right_side.${mesh_ext}"/>
+              <mesh filename="package://robot_properties_bolt/meshes/${mesh_ext}/bolt_upper_leg_left_side.${mesh_ext}"/>
+            </xacro:unless>
+            <xacro:if value="${is_right}">
+              <mesh filename="package://robot_properties_bolt/meshes/${mesh_ext}/bolt_upper_leg_right_side.${mesh_ext}"/>
             </xacro:if>
           </xacro:unless>
           <xacro:if value="${new_leg}">
             <xacro:unless value="${is_right}">
-              <mesh filename="package://meshes/${mesh_ext}/upper_leg_200mm_left_side.${mesh_ext}"/>
-            </xacro:unless>
-            <xacro:if value="${is_right}">
-              <mesh filename="package://meshes/${mesh_ext}/upper_leg_200mm_right_side.${mesh_ext}"/>
+              <mesh filename="package://robot_properties_bolt/meshes/${mesh_ext}/upper_leg_200mm_left_side.${mesh_ext}"/>
+            </xacro:unless>
+            <xacro:if value="${is_right}">
+              <mesh filename="package://robot_properties_bolt/meshes/${mesh_ext}/upper_leg_200mm_right_side.${mesh_ext}"/>
             </xacro:if>
           </xacro:if>
@@ -235,16 +235,16 @@
           <xacro:unless value="${new_leg}">
             <xacro:unless value="${is_right}">
-              <mesh filename="package://meshes/${mesh_ext}/bolt_lower_leg_left_side.${mesh_ext}"/>
-            </xacro:unless>
-            <xacro:if value="${is_right}">
-              <mesh filename="package://meshes/${mesh_ext}/bolt_lower_leg_right_side.${mesh_ext}"/>
+              <mesh filename="package://robot_properties_bolt/meshes/${mesh_ext}/bolt_lower_leg_left_side.${mesh_ext}"/>
+            </xacro:unless>
+            <xacro:if value="${is_right}">
+              <mesh filename="package://robot_properties_bolt/meshes/${mesh_ext}/bolt_lower_leg_right_side.${mesh_ext}"/>
             </xacro:if>
           </xacro:unless>
           <xacro:if value="${new_leg}">
             <xacro:unless value="${is_right}">
-              <mesh filename="package://meshes/${mesh_ext}/lower_leg_200mm_left_side.${mesh_ext}"/>
-            </xacro:unless>
-            <xacro:if value="${is_right}">
-              <mesh filename="package://meshes/${mesh_ext}/lower_leg_200mm_right_side.${mesh_ext}"/>
+              <mesh filename="package://robot_properties_bolt/meshes/${mesh_ext}/lower_leg_200mm_left_side.${mesh_ext}"/>
+            </xacro:unless>
+            <xacro:if value="${is_right}">
+              <mesh filename="package://robot_properties_bolt/meshes/${mesh_ext}/lower_leg_200mm_right_side.${mesh_ext}"/>
             </xacro:if>
           </xacro:if>
@@ -260,16 +260,16 @@
           <xacro:unless value="${new_leg}">
             <xacro:unless value="${is_right}">
-              <mesh filename="package://meshes/${mesh_ext}/bolt_lower_leg_left_side.${mesh_ext}"/>
-            </xacro:unless>
-            <xacro:if value="${is_right}">
-              <mesh filename="package://meshes/${mesh_ext}/bolt_lower_leg_right_side.${mesh_ext}"/>
+              <mesh filename="package://robot_properties_bolt/meshes/${mesh_ext}/bolt_lower_leg_left_side.${mesh_ext}"/>
+            </xacro:unless>
+            <xacro:if value="${is_right}">
+              <mesh filename="package://robot_properties_bolt/meshes/${mesh_ext}/bolt_lower_leg_right_side.${mesh_ext}"/>
             </xacro:if>
           </xacro:unless>
           <xacro:if value="${new_leg}">
             <xacro:unless value="${is_right}">
-              <mesh filename="package://meshes/${mesh_ext}/lower_leg_200mm_left_side.${mesh_ext}"/>
-            </xacro:unless>
-            <xacro:if value="${is_right}">
-              <mesh filename="package://meshes/${mesh_ext}/lower_leg_200mm_right_side.${mesh_ext}"/>
+              <mesh filename="package://robot_properties_bolt/meshes/${mesh_ext}/lower_leg_200mm_left_side.${mesh_ext}"/>
+            </xacro:unless>
+            <xacro:if value="${is_right}">
+              <mesh filename="package://robot_properties_bolt/meshes/${mesh_ext}/lower_leg_200mm_right_side.${mesh_ext}"/>
             </xacro:if>
           </xacro:if>
@@ -315,5 +315,5 @@
         <origin xyz="0 0 0" rpy="0 0 0" />
         <geometry>
-          <mesh filename="package://meshes/${mesh_ext}/bolt_foot.${mesh_ext}"/>
+          <mesh filename="package://robot_properties_bolt/meshes/${mesh_ext}/bolt_foot.${mesh_ext}"/>
         </geometry>
         <material name="${color_name}">
@@ -325,5 +325,5 @@
         <origin xyz="0 0 0" rpy="0 0 0" />
         <geometry>
-          <mesh filename="package://meshes/${mesh_ext}/bolt_foot.${mesh_ext}"/>
+          <mesh filename="package://robot_properties_bolt/meshes/${mesh_ext}/bolt_foot.${mesh_ext}"/>
         </geometry>
         <material name="${color_name}">

File: src/robot_properties_bolt/robot_properties_bolt/xacro/plane_with_restitution.urdf.xacro (robot description, xacro)
@@ -15,5 +15,5 @@
       <origin rpy="0 0 0" xyz="0 0 0"/>
       <geometry>
-      <mesh filename="package://meshes/plane.obj" scale="1 1 1"/>
+      <mesh filename="package://robot_properties_bolt/meshes/plane.obj" scale="1 1 1"/>
       </geometry>
        <material name="white">
