Commit message: first attempt

File: src/robot_properties_bolt/robot_properties_bolt/xacro/bolt_passive_ankle.urdf.xacro (robot description, xacro)
@@ -10,5 +10,5 @@
   <xacro:property name="opacity" value="1.0" />
   <xacro:property name="new_leg" value="true" />
-  <xacro:property name="has_passive_ankle" value="false" />
+  <xacro:property name="has_passive_ankle" value="true" />
   <!-- Include the legs -->
   <xacro:include filename="bolt.xacro"/>

File: src/robot_properties_bolt/robot_properties_bolt/xacro/leg.xacro (robot description, xacro)
@@ -2,5 +2,5 @@
 <robot xmlns:xacro="http://playerstage.sourceforge.net/gazebo/xmlschema/#interface" name="bolt">
   <!-- See TODO: add the wiki link here -->
-  <!-- These are absoulte distance value, the sign are decided below -->
+  <!-- These are absolute distance value, the sign are decided below -->
   <xacro:property name="base_2_HAA_x" value="${0.0 * 0.001}" />
   <xacro:property name="base_2_HAA_y" value="${63.6 * 0.001}" />
@@ -16,5 +16,5 @@
   <!-- Macro defining bolt leg. -->
   <xacro:macro name="leg" params="prefix is_front is_right has_side_motion
-                                  mesh_ext color_name color opacity new_leg">
+                                  mesh_ext color_name color opacity new_leg has_passive_ankle">
     <joint name="${prefix}_HAA" type="revolute">
       <parent link="base_link"/>
@@ -286,5 +286,10 @@
     </link> <!-- END LOWER LEG LINK -->
     <!-- KFE: Joint between the upper leg and the lower leg -->
-    <joint name="${prefix}_ANKLE" type="revolute">
+    <xacro:if value="${has_passive_ankle}">
+      <joint name="${prefix}_ANKLE" type="revolute">
+    </xacro:if>
+    <xacro:unless value="${has_passive_ankle}">
+      <joint name="${prefix}_ANKLE" type="fixed">
+    </xacro:unless>
       <parent link="${prefix}_LOWER_LEG"/>
       <child link="${prefix}_FOOT"/>
@@ -296,6 +301,8 @@
         <origin xyz="0 ${-KFE_2_FOOT_y} ${-KFE_2_FOOT_z}" rpy="0 0 0" />
       </xacro:if>
-      <!-- joints rotates around the y-axis -->
-      <axis xyz="0 1 0"/>
+      <xacro:if value="${has_passive_ankle}">
+        <!-- joints rotates around the y-axis -->
+        <axis xyz="0 1 0"/>
+      </xacro:if>
       <!-- Limits (usefull?) -->
       <limit effort="1000" lower="-10" upper="10" velocity="1000"/>
@@ -308,5 +315,10 @@
       <inertial>
         <origin xyz="0 0 0.00035767" rpy="0 0 0" />
+      <xacro:if value="${has_passive_ankle}">
         <mass value="0.00010"/>
+      </xacro:if>
+      <xacro:unless value="${has_passive_ankle}">
+        <mass value="0.0"/>
+      </xacro:unless>
         <inertia ixx="0.00000057" ixy="0.0"         ixz="0.0"
                  iyy="0.00000084" iyz="0.0"
@@ -315,9 +327,17 @@
       <!-- FOOT VISUAL -->
       <visual>
-<!--        <origin xyz="0 0 0" rpy="0 0 0" />-->
-        <origin xyz="0 0 -0.01" rpy="0 2.35 0" />
-        <geometry>
+      <xacro:if value="${has_passive_ankle}">
+        <origin xyz="0 0 -0.01" rpy="0 2.35 0." />
+      </xacro:if>
+      <xacro:unless value="${has_passive_ankle}">
+        <origin xyz="0 0 0.0" rpy="0 0. 0." />
+      </xacro:unless>
+        <geometry>
+         <xacro:if value="${has_passive_ankle}">
           <cylinder length="0.06" radius="0.0085"/>
-<!--          <mesh filename="package://robot_properties_bolt/meshes/${mesh_ext}/bolt_foot.${mesh_ext}"/>-->
+        </xacro:if>
+        <xacro:unless value="${has_passive_ankle}">
+          <mesh filename="package://robot_properties_bolt/meshes/${mesh_ext}/bolt_foot.${mesh_ext}"/>
+        </xacro:unless>
         </geometry>
         <material name="${color_name}">
@@ -327,9 +347,17 @@
       <!-- FOOT COLLISION -->
       <collision>
+      <xacro:if value="${has_passive_ankle}">
         <origin xyz="0 0 -0.01" rpy="0 2.35 0." />
-<!--        <origin xyz="0 0 0.0" rpy="0 0. 0." />-->
-        <geometry>
+      </xacro:if>
+      <xacro:unless value="${has_passive_ankle}">
+        <origin xyz="0 0 0.0" rpy="0 0. 0." />
+      </xacro:unless>
+        <geometry>
+        <xacro:if value="${has_passive_ankle}">
           <cylinder length="0.06" radius="0.0085"/>
-<!--          <mesh filename="package://robot_properties_bolt/meshes/${mesh_ext}/bolt_foot.${mesh_ext}"/>-->
+        </xacro:if>
+        <xacro:unless value="${has_passive_ankle}">
+          <mesh filename="package://robot_properties_bolt/meshes/${mesh_ext}/bolt_foot.${mesh_ext}"/>
+        </xacro:unless>
         </geometry>
         <material name="${color_name}">
