Commit message: Add Ankle (passive) joint

File: src/robot_properties_bolt/robot_properties_bolt/xacro/leg.xacro (robot description, xacro)
@@ -286,5 +286,5 @@
     </link> <!-- END LOWER LEG LINK -->
     <!-- KFE: Joint between the upper leg and the lower leg -->
-    <joint name="${prefix}_ANKLE" type="fixed">
+    <joint name="${prefix}_ANKLE" type="revolute">
       <parent link="${prefix}_LOWER_LEG"/>
       <child link="${prefix}_FOOT"/>
@@ -296,4 +296,6 @@
         <origin xyz="0 ${-KFE_2_FOOT_y} ${-KFE_2_FOOT_z}" rpy="0 0 0" />
       </xacro:if>
+      <!-- joints rotates around the y-axis -->
+      <axis xyz="0 1 0"/>
       <!-- Limits (usefull?) -->
       <limit effort="1000" lower="-10" upper="10" velocity="1000"/>
@@ -306,5 +308,5 @@
       <inertial>
         <origin xyz="0 0 0.00035767" rpy="0 0 0" />
-        <mass value="0.00000000"/>
+        <mass value="0.00010"/>
         <inertia ixx="0.00000057" ixy="0.0"         ixz="0.0"
                  iyy="0.00000084" iyz="0.0"
@@ -313,7 +315,9 @@
       <!-- FOOT VISUAL -->
       <visual>
-        <origin xyz="0 0 0" rpy="0 0 0" />
-        <geometry>
-          <mesh filename="package://robot_properties_bolt/meshes/${mesh_ext}/bolt_foot.${mesh_ext}"/>
+<!--        <origin xyz="0 0 0" rpy="0 0 0" />-->
+        <origin xyz="0 0 -0.01" rpy="0 2.35 0" />
+        <geometry>
+          <cylinder length="0.06" radius="0.0085"/>
+<!--          <mesh filename="package://robot_properties_bolt/meshes/${mesh_ext}/bolt_foot.${mesh_ext}"/>-->
         </geometry>
         <material name="${color_name}">
@@ -323,7 +327,9 @@
       <!-- FOOT COLLISION -->
       <collision>
-        <origin xyz="0 0 0" rpy="0 0 0" />
-        <geometry>
-          <mesh filename="package://robot_properties_bolt/meshes/${mesh_ext}/bolt_foot.${mesh_ext}"/>
+        <origin xyz="0 0 -0.01" rpy="0 2.35 0." />
+<!--        <origin xyz="0 0 0.0" rpy="0 0. 0." />-->
+        <geometry>
+          <cylinder length="0.06" radius="0.0085"/>
+<!--          <mesh filename="package://robot_properties_bolt/meshes/${mesh_ext}/bolt_foot.${mesh_ext}"/>-->
         </geometry>
         <material name="${color_name}">

Commit message: fix usage of the passive ankle in simulation

File: src/robot_properties_bolt/robot_properties_bolt/xacro/leg.xacro (robot description, xacro)
@@ -1,34 +1,41 @@
 <?xml version="1.0"?>
 <robot xmlns:xacro="http://playerstage.sourceforge.net/gazebo/xmlschema/#interface" name="bolt">
-  <!-- See TODO: add the wiki link here -->
-  <!-- These are absolute distance value, the sign are decided below -->
-  <xacro:property name="base_2_HAA_x" value="${0.0 * 0.001}" />
-  <xacro:property name="base_2_HAA_y" value="${63.6 * 0.001}" />
-  <!--xacro:property name="base_2_HAA_x" value="${2.45656 * 0.001}" />
+<!-- See TODO: add the wiki link here -->
+<!-- These are absolute distance value, the sign are decided below -->
+    <xacro:property name="base_2_HAA_x" value="${0.0 * 0.001}" />
+    <xacro:property name="base_2_HAA_y" value="${63.6 * 0.001}" />
+    <!--xacro:property name="base_2_HAA_x" value="${2.45656 * 0.001}" />
   <xacro:property name="base_2_HAA_y" value="${63.6 * 0.001}" />
   <xacro:property name="base_2_HAA_z" value="${33.0809 * 0.001}" /-->
-  <xacro:property name="HAA_2_HFE_y" value="${14.5 * 0.001}" />
-  <xacro:property name="HAA_2_HFE_z" value="${38.60 * 0.001}" />
-  <xacro:property name="HFE_2_KFE_y" value="${37.4 * 0.001}" />
-  <xacro:property name="HFE_2_KFE_z" value="${200.00 * 0.001}" />
-  <xacro:property name="KFE_2_FOOT_y" value="${8.0 * 0.001}" />
-  <xacro:property name="KFE_2_FOOT_z" value="${200.00 * 0.001}" />
-  <!-- Macro defining bolt leg. -->
-  <xacro:macro name="leg" params="prefix is_front is_right has_side_motion
-                                  mesh_ext color_name color opacity new_leg has_passive_ankle">
-    <joint name="${prefix}_HAA" type="revolute">
-      <parent link="base_link"/>
-      <child link="${prefix}_SHOULDER"/>
-      <limit effort="1000" lower="-10" upper="10" velocity="1000"/>
-      <!-- joints rotates around the x-axis -->
-      <axis xyz="1 0 0"/>
-      <!-- placement of the joint -->
-      <xacro:unless value="${is_right}">
-        <origin xyz="${base_2_HAA_x} ${base_2_HAA_y} 0" rpy="0 0 0" />
-      </xacro:unless>
-      <xacro:if value="${is_right}">
-        <origin xyz="${base_2_HAA_x} ${-base_2_HAA_y} 0" rpy="0 0 0" />
-      </xacro:if>
-      <!--xacro:unless value="${is_right}">
+    <xacro:property name="HAA_2_HFE_y" value="${14.5 * 0.001}" />
+    <xacro:property name="HAA_2_HFE_z" value="${38.60 * 0.001}" />
+    <xacro:property name="HFE_2_KFE_y" value="${37.4 * 0.001}" />
+    <xacro:property name="HFE_2_KFE_z" value="${200.00 * 0.001}" />
+    <xacro:property name="KFE_2_FOOT_y" value="${8.0 * 0.001}" />
+    <xacro:property name="KFE_2_FOOT_z" value="${200.00 * 0.001}" />
+    <xacro:if value="${has_passive_ankle}">
+        <xacro:property name="ankle_joint_type" value="revolute" />
+    </xacro:if>
+    <xacro:unless value="${has_passive_ankle}">
+        <xacro:property name="ankle_joint_type" value="fixed" />
+    </xacro:unless>
+    <!-- Macro defining bolt leg. -->
+    <xacro:macro name="leg" params="prefix is_front is_right has_side_motion
+                                    mesh_ext color_name color opacity new_leg
+                                    has_passive_ankle">
+        <joint name="${prefix}_HAA" type="revolute">
+            <parent link="base_link"/>
+            <child link="${prefix}_SHOULDER"/>
+            <limit effort="1000" lower="-10" upper="10" velocity="1000"/>
+            <!-- joints rotates around the x-axis -->
+            <axis xyz="1 0 0"/>
+            <!-- placement of the joint -->
+            <xacro:unless value="${is_right}">
+                <origin xyz="${base_2_HAA_x} ${base_2_HAA_y} 0" rpy="0 0 0"/>
+            </xacro:unless>
+            <xacro:if value="${is_right}">
+                <origin xyz="${base_2_HAA_x} ${-base_2_HAA_y} 0" rpy="0 0 0"/>
+            </xacro:if>
+            <!--xacro:unless value="${is_right}">
         <origin xyz="${base_2_HAA_x} ${base_2_HAA_y + 0.0007888} ${-base_2_HAA_z}" rpy="0 0 0" />
       </xacro:unless>
@@ -36,339 +43,358 @@
         <origin xyz="${base_2_HAA_x} ${-base_2_HAA_y + 0.0007888} ${-base_2_HAA_z}" rpy="0 0 0" />
       </xacro:if-->
-      <!-- pybullet simulation parameters -->
-      <dynamics damping="0.0" friction="0.0"/>
-    </joint>
-    <link name="${prefix}_SHOULDER">
-      <!-- TODO: Update inertias and add visuals for link. -->
-      <!-- create a dummy shoulder link to join the two joints -->
-      <inertial>
-        <xacro:unless value="${is_right}">
-          <!-- Left upper leg inertia -->
-          <mass value="0.14004265"/>
-          <origin xyz="0.01708256 -0.00446892 -0.01095830" rpy="0 0 0" />
-          <inertia ixx="0.00007443" ixy="0.00000148" ixz="0.00002154"
-                   iyy="0.00013847" iyz="-0.00001096"
-                   izz="0.00009002"/>
-        </xacro:unless>
-        <xacro:if value="${is_right}">
-          <!-- Right upper leg inertia -->
-          <mass value="0.14004412"/>
-          <origin xyz="0.01708233 0.00447099 -0.01095846" rpy="0 0 0" />
-          <inertia ixx="0.00007442" ixy="-0.00000148" ixz="0.00002154"
-                   iyy="0.00013848"  iyz="0.00001095"
-                   izz="0.00009001"/>
-        </xacro:if>
-      </inertial>
-      <!-- HIP LEG LINK VISUAL -->
-      <visual>
-        <origin xyz="0 0 0" rpy="0 0 0" />
-        <geometry>
-          <xacro:unless value="${is_right}">
-            <mesh filename="package://robot_properties_bolt/meshes/${mesh_ext}/bolt_hip_fe_left_side.${mesh_ext}"/>
-          </xacro:unless>
-          <xacro:if value="${is_right}">
-            <mesh filename="package://robot_properties_bolt/meshes/${mesh_ext}/bolt_hip_fe_right_side.${mesh_ext}"/>
-          </xacro:if>
-        </geometry>
-        <material name="${color_name}">
-          <color rgba="${color} ${opacity}"/>
-        </material>
-      </visual>
-      <!-- UPPER LEG LINK COLLISION -->
-      <collision>
-        <origin xyz="0 0 0" rpy="0 0 0" />
-        <geometry>
-          <xacro:unless value="${is_right}">
-            <mesh filename="package://robot_properties_bolt/meshes/${mesh_ext}/bolt_hip_fe_left_side.${mesh_ext}"/>
-          </xacro:unless>
-          <xacro:if value="${is_right}">
-            <mesh filename="package://robot_properties_bolt/meshes/${mesh_ext}/bolt_hip_fe_right_side.${mesh_ext}"/>
-          </xacro:if>
-        </geometry>
-        <material name="${color_name}">
-          <color rgba="${color} ${opacity}"/>
-        </material>
-      </collision>
-      <!-- Bullet specific paramters -->
-      <contact>
-        <lateral_friction value="1.0"/>
-        <restitution value="0.5"/>
-      </contact>
-    </link>
-    <joint name="${prefix}_HFE" type="revolute">
-      <parent link="${prefix}_SHOULDER"/>
-      <child link="${prefix}_UPPER_LEG"/>
-      <limit effort="1000" lower="-10" upper="10" velocity="1000"/>
-      <!-- joints rotates around the y-axis -->
-      <axis xyz="0 1 0"/>
-      <!-- placement of the joint -->
-      <xacro:if value="${is_right}">
-        <origin xyz="0 ${-HAA_2_HFE_y} ${-HAA_2_HFE_z}" rpy="0 0 0" />
-      </xacro:if>
-      <xacro:unless value="${is_right}">
-        <origin xyz="0 ${HAA_2_HFE_y} ${-HAA_2_HFE_z}" rpy="0 0 0" />
-      </xacro:unless>
-      <!-- pybullet simulation parameters -->
-      <dynamics damping="0.0" friction="0.0"/>
-    </joint>
-    <link name="${prefix}_UPPER_LEG">
-      <!-- UPPER LEG LINK INERTIAL -->
-      <xacro:unless value="${is_right}">
-        <!-- Left upper leg inertia -->
-        <inertial>
-          <origin xyz="0.00001377 0.01935853 -0.11870700" rpy="0 0 0" />
-          <mass value="0.14853845"/>
-          <inertia ixx="0.00041107" ixy="0.00000000"  ixz="0.00000009"
-                   iyy="0.00041193"  iyz="-0.00004671"
-                   izz="0.00003024"/>
-        </inertial>
-      </xacro:unless>
-      <xacro:if value="${is_right}">
-        <!-- Right upper leg inertia -->
-        <inertial>
-          <origin xyz="-0.00001377 -0.01935853 -0.11870700" rpy="0 0 0" />
-          <mass value="0.14853845"/>
-          <inertia ixx="0.00041107" ixy="0.00000000"  ixz="-0.00000009"
-                   iyy="0.00041193"  iyz="0.00004671"
-                   izz="0.00003024"/>
-        </inertial>
-      </xacro:if>
-      <!-- UPPER LEG LINK VISUAL -->
-      <visual>
-        <origin xyz="0 0 0" rpy="0 0 0" />
-        <geometry>
-          <xacro:unless value="${new_leg}">
-            <xacro:unless value="${is_right}">
-              <mesh filename="package://robot_properties_bolt/meshes/${mesh_ext}/bolt_upper_leg_left_side.${mesh_ext}"/>
-            </xacro:unless>
-            <xacro:if value="${is_right}">
-              <mesh filename="package://robot_properties_bolt/meshes/${mesh_ext}/bolt_upper_leg_right_side.${mesh_ext}"/>
-            </xacro:if>
-          </xacro:unless>
-          <xacro:if value="${new_leg}">
-            <xacro:unless value="${is_right}">
-              <mesh filename="package://robot_properties_bolt/meshes/${mesh_ext}/upper_leg_200mm_left_side.${mesh_ext}"/>
-            </xacro:unless>
-            <xacro:if value="${is_right}">
-              <mesh filename="package://robot_properties_bolt/meshes/${mesh_ext}/upper_leg_200mm_right_side.${mesh_ext}"/>
-            </xacro:if>
-          </xacro:if>
-        </geometry>
-        <material name="${color_name}">
-          <color rgba="${color} ${opacity}"/>
-        </material>
-      </visual>
-      <!-- UPPER LEG LINK COLLISION -->
-      <collision>
-        <origin xyz="0 0 0" rpy="0 0 0" />
-        <geometry>
-          <xacro:unless value="${new_leg}">
-            <xacro:unless value="${is_right}">
-              <mesh filename="package://robot_properties_bolt/meshes/${mesh_ext}/bolt_upper_leg_left_side.${mesh_ext}"/>
-            </xacro:unless>
-            <xacro:if value="${is_right}">
-              <mesh filename="package://robot_properties_bolt/meshes/${mesh_ext}/bolt_upper_leg_right_side.${mesh_ext}"/>
-            </xacro:if>
-          </xacro:unless>
-          <xacro:if value="${new_leg}">
-            <xacro:unless value="${is_right}">
-              <mesh filename="package://robot_properties_bolt/meshes/${mesh_ext}/upper_leg_200mm_left_side.${mesh_ext}"/>
-            </xacro:unless>
-            <xacro:if value="${is_right}">
-              <mesh filename="package://robot_properties_bolt/meshes/${mesh_ext}/upper_leg_200mm_right_side.${mesh_ext}"/>
-            </xacro:if>
-          </xacro:if>
-        </geometry>
-        <material name="${color_name}">
-          <color rgba="${color} ${opacity}"/>
-        </material>
-      </collision>
-      <!-- Bullet specific paramters -->
-      <contact>
-        <lateral_friction value="1.0"/>
-        <restitution value="0.5"/>
-      </contact>
-    </link> <!-- END UPPER LEG LINK -->
-    <!-- KFE: Joint between the upper leg and the lower leg -->
-    <joint name="${prefix}_KFE" type="revolute">
-      <parent link="${prefix}_UPPER_LEG"/>
-      <child link="${prefix}_LOWER_LEG"/>
-      <limit effort="1000" lower="-10" upper="10" velocity="1000"/>
-      <!-- joints rotates around the y-axis -->
-      <axis xyz="0 1 0"/>
-      <!-- placement of the joint -->
-      <xacro:unless value="${is_right}">
-        <origin xyz="0 ${HFE_2_KFE_y} ${-HFE_2_KFE_z}" rpy="0 0 0" />
-      </xacro:unless>
-      <xacro:if value="${is_right}">
-        <origin xyz="0 ${-HFE_2_KFE_y} ${-HFE_2_KFE_z}" rpy="0 0 0" />
-      </xacro:if>
-      <!-- pybullet simulation parameters -->
-      <dynamics damping="0.0" friction="0.0"/>
-    </joint>
-    <link name="${prefix}_LOWER_LEG">
-      <!-- LOWER LEG LINK INERTIAL -->
-      <xacro:unless value="${is_right}">
-        <!-- Left lower leg inertia -->
-        <inertial>
-          <origin xyz="0.0 0.00836718 -0.11591877" rpy="0 0 0" />
-          <mass value="0.03117243"/>
-          <inertia ixx="0.00011487" ixy="0.00000000"  ixz="0.00000000"
-                   iyy="0.00011556"  iyz="-0.00000190"
-                   izz="0.00000220"/>
-        </inertial>
-      </xacro:unless>
-      <xacro:if value="${is_right}">
-        <!-- Right lower leg inertia -->
-        <inertial>
-          <origin xyz="0.0 -0.00836718 -0.11591877" rpy="0 0 0" />
-          <mass value="0.03117243"/>
-          <inertia ixx="0.00011487" ixy="0.00000000"  ixz="0.00000000"
-                   iyy="0.00011556"  iyz="0.00000190"
-                   izz="0.00000220"/>
-        </inertial>
-      </xacro:if>
-      <!-- LOWER LEG LINK VISUAL -->
-      <visual>
-        <origin xyz="0 0 0" rpy="0 0 0" />
-        <geometry>
-          <xacro:unless value="${new_leg}">
-            <xacro:unless value="${is_right}">
-              <mesh filename="package://robot_properties_bolt/meshes/${mesh_ext}/bolt_lower_leg_left_side.${mesh_ext}"/>
-            </xacro:unless>
-            <xacro:if value="${is_right}">
-              <mesh filename="package://robot_properties_bolt/meshes/${mesh_ext}/bolt_lower_leg_right_side.${mesh_ext}"/>
-            </xacro:if>
-          </xacro:unless>
-          <xacro:if value="${new_leg}">
-            <xacro:unless value="${is_right}">
-              <mesh filename="package://robot_properties_bolt/meshes/${mesh_ext}/lower_leg_200mm_left_side.${mesh_ext}"/>
-            </xacro:unless>
-            <xacro:if value="${is_right}">
-              <mesh filename="package://robot_properties_bolt/meshes/${mesh_ext}/lower_leg_200mm_right_side.${mesh_ext}"/>
-            </xacro:if>
-          </xacro:if>
-        </geometry>
-        <material name="${color_name}">
-          <color rgba="${color} ${opacity}"/>
-        </material>
-      </visual>
-      <!-- LOWER LEG LINK COLLISION -->
-      <collision>
-        <origin xyz="0 0 0" rpy="0 0 0" />
-        <geometry>
-          <xacro:unless value="${new_leg}">
-            <xacro:unless value="${is_right}">
-              <mesh filename="package://robot_properties_bolt/meshes/${mesh_ext}/bolt_lower_leg_left_side.${mesh_ext}"/>
-            </xacro:unless>
-            <xacro:if value="${is_right}">
-              <mesh filename="package://robot_properties_bolt/meshes/${mesh_ext}/bolt_lower_leg_right_side.${mesh_ext}"/>
-            </xacro:if>
-          </xacro:unless>
-          <xacro:if value="${new_leg}">
-            <xacro:unless value="${is_right}">
-              <mesh filename="package://robot_properties_bolt/meshes/${mesh_ext}/lower_leg_200mm_left_side.${mesh_ext}"/>
-            </xacro:unless>
-            <xacro:if value="${is_right}">
-              <mesh filename="package://robot_properties_bolt/meshes/${mesh_ext}/lower_leg_200mm_right_side.${mesh_ext}"/>
-            </xacro:if>
-          </xacro:if>
-        </geometry>
-        <material name="${color_name}">
-          <color rgba="${color} ${opacity}"/>
-        </material>
-      </collision>
-      <!-- Bullet specific paramters -->
-      <contact>
-        <lateral_friction value="1.0"/>
-        <restitution value="0.5"/>
-      </contact>
-    </link> <!-- END LOWER LEG LINK -->
-    <!-- KFE: Joint between the upper leg and the lower leg -->
-    <xacro:if value="${has_passive_ankle}">
-      <joint name="${prefix}_ANKLE" type="revolute">
-    </xacro:if>
-    <xacro:unless value="${has_passive_ankle}">
-      <joint name="${prefix}_ANKLE" type="fixed">
-    </xacro:unless>
-      <parent link="${prefix}_LOWER_LEG"/>
-      <child link="${prefix}_FOOT"/>
-      <!-- Joint placement -->
-      <xacro:unless value="${is_right}">
-        <origin xyz="0 ${KFE_2_FOOT_y} ${-KFE_2_FOOT_z}" rpy="0 0 0" />
-      </xacro:unless>
-      <xacro:if value="${is_right}">
-        <origin xyz="0 ${-KFE_2_FOOT_y} ${-KFE_2_FOOT_z}" rpy="0 0 0" />
-      </xacro:if>
-      <xacro:if value="${has_passive_ankle}">
-        <!-- joints rotates around the y-axis -->
-        <axis xyz="0 1 0"/>
-      </xacro:if>
-      <!-- Limits (usefull?) -->
-      <limit effort="1000" lower="-10" upper="10" velocity="1000"/>
-      <!-- pybullet simulation parameters -->
-      <dynamics damping="0.0" friction="0.0"/>
-    </joint>
-    <link name="${prefix}_FOOT">
-      <!-- FOOT INERTIAL -->
-      <!-- This link is symmetrical left or right -->
-      <inertial>
-        <origin xyz="0 0 0.00035767" rpy="0 0 0" />
-      <xacro:if value="${has_passive_ankle}">
-        <mass value="0.00010"/>
-      </xacro:if>
-      <xacro:unless value="${has_passive_ankle}">
-        <mass value="0.0"/>
-      </xacro:unless>
-        <inertia ixx="0.00000057" ixy="0.0"         ixz="0.0"
-                 iyy="0.00000084" iyz="0.0"
-                 izz="0.00000053"/>
-      </inertial>
-      <!-- FOOT VISUAL -->
-      <visual>
-      <xacro:if value="${has_passive_ankle}">
-        <origin xyz="0 0 -0.01" rpy="0 2.35 0." />
-      </xacro:if>
-      <xacro:unless value="${has_passive_ankle}">
-        <origin xyz="0 0 0.0" rpy="0 0. 0." />
-      </xacro:unless>
-        <geometry>
-         <xacro:if value="${has_passive_ankle}">
-          <cylinder length="0.06" radius="0.0085"/>
-        </xacro:if>
-        <xacro:unless value="${has_passive_ankle}">
-          <mesh filename="package://robot_properties_bolt/meshes/${mesh_ext}/bolt_foot.${mesh_ext}"/>
-        </xacro:unless>
-        </geometry>
-        <material name="${color_name}">
-          <color rgba="${color} ${opacity}"/>
-        </material>
-      </visual>
-      <!-- FOOT COLLISION -->
-      <collision>
-      <xacro:if value="${has_passive_ankle}">
-        <origin xyz="0 0 -0.01" rpy="0 2.35 0." />
-      </xacro:if>
-      <xacro:unless value="${has_passive_ankle}">
-        <origin xyz="0 0 0.0" rpy="0 0. 0." />
-      </xacro:unless>
-        <geometry>
-        <xacro:if value="${has_passive_ankle}">
-          <cylinder length="0.06" radius="0.0085"/>
-        </xacro:if>
-        <xacro:unless value="${has_passive_ankle}">
-          <mesh filename="package://robot_properties_bolt/meshes/${mesh_ext}/bolt_foot.${mesh_ext}"/>
-        </xacro:unless>
-        </geometry>
-        <material name="${color_name}">
-          <color rgba="${color} ${opacity}"/>
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