Commit message: rename the 'robot_porperties_bolt' folder as 'resources'

File: src/robot_properties_bolt/resources/xacro/bolt.xacro (robot description, xacro)
@@ -22,5 +22,5 @@
           <origin xyz="0 0 0" rpy="0 0 0" />
           <geometry>
-            <mesh filename="package://robot_properties_bolt/meshes/${mesh_ext}/bolt_body.${mesh_ext}"/>
+            <mesh filename="package://robot_properties_bolt/resources/meshes/${mesh_ext}/bolt_body.${mesh_ext}"/>
           </geometry>
           <material name="${color_name}">
@@ -32,5 +32,5 @@
           <origin xyz="0 0 0" rpy="0 0 0" />
           <geometry>
-            <mesh filename="package://robot_properties_bolt/meshes/${mesh_ext}/bolt_body.${mesh_ext}"/>
+            <mesh filename="package://robot_properties_bolt/resources/meshes/${mesh_ext}/bolt_body.${mesh_ext}"/>
           </geometry>
           <material name="${color_name}">

File: src/robot_properties_bolt/resources/xacro/leg.xacro (robot description, xacro)
@@ -78,8 +78,8 @@
                 <geometry>
                     <xacro:unless value="${is_right}">
-                        <mesh filename="package://robot_properties_bolt/meshes/${mesh_ext}/bolt_hip_fe_left_side.${mesh_ext}"/>
+                        <mesh filename="package://robot_properties_bolt/resources/meshes/${mesh_ext}/bolt_hip_fe_left_side.${mesh_ext}"/>
                     </xacro:unless>
                     <xacro:if value="${is_right}">
-                        <mesh filename="package://robot_properties_bolt/meshes/${mesh_ext}/bolt_hip_fe_right_side.${mesh_ext}"/>
+                        <mesh filename="package://robot_properties_bolt/resources/meshes/${mesh_ext}/bolt_hip_fe_right_side.${mesh_ext}"/>
                     </xacro:if>
                 </geometry>
@@ -93,8 +93,8 @@
                 <geometry>
                     <xacro:unless value="${is_right}">
-                        <mesh filename="package://robot_properties_bolt/meshes/${mesh_ext}/bolt_hip_fe_left_side.${mesh_ext}"/>
+                        <mesh filename="package://robot_properties_bolt/resources/meshes/${mesh_ext}/bolt_hip_fe_left_side.${mesh_ext}"/>
                     </xacro:unless>
                     <xacro:if value="${is_right}">
-                        <mesh filename="package://robot_properties_bolt/meshes/${mesh_ext}/bolt_hip_fe_right_side.${mesh_ext}"/>
+                        <mesh filename="package://robot_properties_bolt/resources/meshes/${mesh_ext}/bolt_hip_fe_right_side.${mesh_ext}"/>
                     </xacro:if>
                 </geometry>
@@ -159,16 +159,16 @@
                     <xacro:unless value="${new_leg}">
                         <xacro:unless value="${is_right}">
-                            <mesh filename="package://robot_properties_bolt/meshes/${mesh_ext}/bolt_upper_leg_left_side.${mesh_ext}"/>
-                        </xacro:unless>
-                        <xacro:if value="${is_right}">
-                            <mesh filename="package://robot_properties_bolt/meshes/${mesh_ext}/bolt_upper_leg_right_side.${mesh_ext}"/>
+                            <mesh filename="package://robot_properties_bolt/resources/meshes/${mesh_ext}/bolt_upper_leg_left_side.${mesh_ext}"/>
+                        </xacro:unless>
+                        <xacro:if value="${is_right}">
+                            <mesh filename="package://robot_properties_bolt/resources/meshes/${mesh_ext}/bolt_upper_leg_right_side.${mesh_ext}"/>
                         </xacro:if>
                     </xacro:unless>
                     <xacro:if value="${new_leg}">
                         <xacro:unless value="${is_right}">
-                            <mesh filename="package://robot_properties_bolt/meshes/${mesh_ext}/upper_leg_200mm_left_side.${mesh_ext}"/>
-                        </xacro:unless>
-                        <xacro:if value="${is_right}">
-                            <mesh filename="package://robot_properties_bolt/meshes/${mesh_ext}/upper_leg_200mm_right_side.${mesh_ext}"/>
+                            <mesh filename="package://robot_properties_bolt/resources/meshes/${mesh_ext}/upper_leg_200mm_left_side.${mesh_ext}"/>
+                        </xacro:unless>
+                        <xacro:if value="${is_right}">
+                            <mesh filename="package://robot_properties_bolt/resources/meshes/${mesh_ext}/upper_leg_200mm_right_side.${mesh_ext}"/>
                         </xacro:if>
                     </xacro:if>
@@ -184,16 +184,16 @@
                     <xacro:unless value="${new_leg}">
                         <xacro:unless value="${is_right}">
-                            <mesh filename="package://robot_properties_bolt/meshes/${mesh_ext}/bolt_upper_leg_left_side.${mesh_ext}"/>
-                        </xacro:unless>
-                        <xacro:if value="${is_right}">
-                            <mesh filename="package://robot_properties_bolt/meshes/${mesh_ext}/bolt_upper_leg_right_side.${mesh_ext}"/>
+                            <mesh filename="package://robot_properties_bolt/resources/meshes/${mesh_ext}/bolt_upper_leg_left_side.${mesh_ext}"/>
+                        </xacro:unless>
+                        <xacro:if value="${is_right}">
+                            <mesh filename="package://robot_properties_bolt/resources/meshes/${mesh_ext}/bolt_upper_leg_right_side.${mesh_ext}"/>
                         </xacro:if>
                     </xacro:unless>
                     <xacro:if value="${new_leg}">
                         <xacro:unless value="${is_right}">
-                            <mesh filename="package://robot_properties_bolt/meshes/${mesh_ext}/upper_leg_200mm_left_side.${mesh_ext}"/>
-                        </xacro:unless>
-                        <xacro:if value="${is_right}">
-                            <mesh filename="package://robot_properties_bolt/meshes/${mesh_ext}/upper_leg_200mm_right_side.${mesh_ext}"/>
+                            <mesh filename="package://robot_properties_bolt/resources/meshes/${mesh_ext}/upper_leg_200mm_left_side.${mesh_ext}"/>
+                        </xacro:unless>
+                        <xacro:if value="${is_right}">
+                            <mesh filename="package://robot_properties_bolt/resources/meshes/${mesh_ext}/upper_leg_200mm_right_side.${mesh_ext}"/>
                         </xacro:if>
                     </xacro:if>
@@ -261,16 +261,16 @@
                     <xacro:unless value="${new_leg}">
                         <xacro:unless value="${is_right}">
-                            <mesh filename="package://robot_properties_bolt/meshes/${mesh_ext}/bolt_lower_leg_left_side.${mesh_ext}"/>
-                        </xacro:unless>
-                        <xacro:if value="${is_right}">
-                            <mesh filename="package://robot_properties_bolt/meshes/${mesh_ext}/bolt_lower_leg_right_side.${mesh_ext}"/>
+                            <mesh filename="package://robot_properties_bolt/resources/meshes/${mesh_ext}/bolt_lower_leg_left_side.${mesh_ext}"/>
+                        </xacro:unless>
+                        <xacro:if value="${is_right}">
+                            <mesh filename="package://robot_properties_bolt/resources/meshes/${mesh_ext}/bolt_lower_leg_right_side.${mesh_ext}"/>
                         </xacro:if>
                     </xacro:unless>
                     <xacro:if value="${new_leg}">
                         <xacro:unless value="${is_right}">
-                            <mesh filename="package://robot_properties_bolt/meshes/${mesh_ext}/lower_leg_200mm_left_side.${mesh_ext}"/>
-                        </xacro:unless>
-                        <xacro:if value="${is_right}">
-                            <mesh filename="package://robot_properties_bolt/meshes/${mesh_ext}/lower_leg_200mm_right_side.${mesh_ext}"/>
+                            <mesh filename="package://robot_properties_bolt/resources/meshes/${mesh_ext}/lower_leg_200mm_left_side.${mesh_ext}"/>
+                        </xacro:unless>
+                        <xacro:if value="${is_right}">
+                            <mesh filename="package://robot_properties_bolt/resources/meshes/${mesh_ext}/lower_leg_200mm_right_side.${mesh_ext}"/>
                         </xacro:if>
                     </xacro:if>
@@ -286,16 +286,16 @@
                     <xacro:unless value="${new_leg}">
                         <xacro:unless value="${is_right}">
-                            <mesh filename="package://robot_properties_bolt/meshes/${mesh_ext}/bolt_lower_leg_left_side.${mesh_ext}"/>
-                        </xacro:unless>
-                        <xacro:if value="${is_right}">
-                            <mesh filename="package://robot_properties_bolt/meshes/${mesh_ext}/bolt_lower_leg_right_side.${mesh_ext}"/>
+                            <mesh filename="package://robot_properties_bolt/resources/meshes/${mesh_ext}/bolt_lower_leg_left_side.${mesh_ext}"/>
+                        </xacro:unless>
+                        <xacro:if value="${is_right}">
+                            <mesh filename="package://robot_properties_bolt/resources/meshes/${mesh_ext}/bolt_lower_leg_right_side.${mesh_ext}"/>
                         </xacro:if>
                     </xacro:unless>
                     <xacro:if value="${new_leg}">
                         <xacro:unless value="${is_right}">
-                            <mesh filename="package://robot_properties_bolt/meshes/${mesh_ext}/lower_leg_200mm_left_side.${mesh_ext}"/>
-                        </xacro:unless>
-                        <xacro:if value="${is_right}">
-                            <mesh filename="package://robot_properties_bolt/meshes/${mesh_ext}/lower_leg_200mm_right_side.${mesh_ext}"/>
+                            <mesh filename="package://robot_properties_bolt/resources/meshes/${mesh_ext}/lower_leg_200mm_left_side.${mesh_ext}"/>
+                        </xacro:unless>
+                        <xacro:if value="${is_right}">
+                            <mesh filename="package://robot_properties_bolt/resources/meshes/${mesh_ext}/lower_leg_200mm_right_side.${mesh_ext}"/>
                         </xacro:if>
                     </xacro:if>
@@ -363,5 +363,5 @@
                     </xacro:if>
                     <xacro:unless value="${has_passive_ankle}">
-                        <mesh filename="package://robot_properties_bolt/meshes/${mesh_ext}/bolt_foot.${mesh_ext}"/>
+                        <mesh filename="package://robot_properties_bolt/resources/meshes/${mesh_ext}/bolt_foot.${mesh_ext}"/>
                     </xacro:unless>
                 </geometry>
@@ -383,5 +383,5 @@
                     </xacro:if>
                     <xacro:unless value="${has_passive_ankle}">
-                        <mesh filename="package://robot_properties_bolt/meshes/${mesh_ext}/bolt_foot.${mesh_ext}"/>
+                        <mesh filename="package://robot_properties_bolt/resources/meshes/${mesh_ext}/bolt_foot.${mesh_ext}"/>
                     </xacro:unless>
                 </geometry>

File: src/robot_properties_bolt/resources/xacro/plane_with_restitution.urdf.xacro (robot description, xacro)
@@ -15,5 +15,5 @@
       <origin rpy="0 0 0" xyz="0 0 0"/>
       <geometry>
-      <mesh filename="package://robot_properties_bolt/meshes/plane.obj" scale="1 1 1"/>
+      <mesh filename="package://robot_properties_bolt/resources/meshes/plane.obj" scale="1 1 1"/>
       </geometry>
        <material name="white">
