Commit message: Set active_ankle as default joint + change urdf parameters

File: src/robot_properties_bolt/resources/xacro/leg.xacro (robot description, xacro)
@@ -323,8 +323,6 @@
                 <origin xyz="0 ${-KFE_2_FOOT_y} ${-KFE_2_FOOT_z}" rpy="0 0 0"/>
             </xacro:if>
-            <xacro:if value="${has_passive_ankle}">
             <!-- joints rotates around the y-axis -->
-                <axis xyz="0 1 0"/>
-            </xacro:if>
+            <axis xyz="0 1 0"/>
             <!-- Limits (usefull?) -->
             <limit effort="1000" lower="-10" upper="10" velocity="1000"/>
@@ -337,10 +335,5 @@
             <inertial>
                 <origin xyz="0 0 0.00035767" rpy="0 0 0"/>
-                <xacro:if value="${has_passive_ankle}">
-                    <mass value="0.00010"/>
-                </xacro:if>
-                <xacro:unless value="${has_passive_ankle}">
-                    <mass value="0.0"/>
-                </xacro:unless>
+                <mass value="0.00010"/>
                 <inertia ixx="0.00000057"
                     ixy="0.0"
@@ -352,10 +345,5 @@
             <!-- FOOT VISUAL -->
             <visual>
-                <xacro:if value="${has_passive_ankle}">
-                    <origin xyz="0 0 -0.01" rpy="0 2.35 0."/>
-                </xacro:if>
-                <xacro:unless value="${has_passive_ankle}">
-                    <origin xyz="0 0 0.0" rpy="0 0. 0."/>
-                </xacro:unless>
+                <origin xyz="0 0 -0.01" rpy="0 2.35 0."/>
                 <geometry>
                     <xacro:if value="${has_passive_ankle}">
@@ -372,10 +360,5 @@
             <!-- FOOT COLLISION -->
             <collision>
-                <xacro:if value="${has_passive_ankle}">
-                    <origin xyz="0 0 -0.01" rpy="0 2.35 0."/>
-                </xacro:if>
-                <xacro:unless value="${has_passive_ankle}">
-                    <origin xyz="0 0 0.0" rpy="0 0. 0."/>
-                </xacro:unless>
+                <origin xyz="0 0 -0.01" rpy="0 2.35 0."/>
                 <geometry>
                     <xacro:if value="${has_passive_ankle}">
