Commit message: construct upper body xacro file

File: src/robot_properties_bolt/resources/xacro/bolt_humanoid.xacro (robot description, xacro)
@@ -6,7 +6,7 @@
   xmlns:xacro="http://playerstage.sourceforge.net/gazebo/xmlschema/#interface">
   <xacro:macro name="bolt_full" params="mesh_ext color_name color opacity new_leg has_passive_ankle">
-    <!-- This file is based on: https://atlas.is.localnet/confluence/display/AMDW/Quadruped+URDF+Files -->
+    <!-- This file is based on:  -->
     <link name="base_link">
-      <!-- BASE LINK INERTIAL -->
+      <!-- BASE LINK INERTIA -->
       <inertial>
           <origin xyz="0 0 0" rpy="0 0 0" />

File: src/robot_properties_bolt/resources/xacro/upper_body.xacro (robot description, xacro)
@@ -1,6 +1,140 @@
 <?xml version="1.0"?>
 <robot xmlns:xacro="http://playerstage.sourceforge.net/gazebo/xmlschema/#interface" name="bolt">
-    <!-- These are absolute distance value, the sign are decided below -->
-    <!-- WA stands for Waist Yaw joint, SFE is shoulder flexion-extension -->
-    <xacro:property name="base_2_WY_z" value="${76.0 * 0.001}" />
+  <!-- These are absolute distance value, the sign are decided below -->
+  <!-- WA stands for Waist Rotation joint, SFE is shoulder flexion-extension -->
+  <xacro:property name="base_2_WR_z" value="${76.0 * 0.001}" />
+  <xacro:property name="WR_2_SFE_y" value="${110.0 * 0.001}" />
+  <xacro:property name="WR_2_SFE_z" value="${160.0 * 0.001}" />
+  <!-- Macro defining bolt upper_body. -->
+  <xacro:macro name="upper_body" params="prefix is_right has_side_motion mesh_ext color_name color">
+    <joint name="${prefix}_WR" type="revolute">
+        <parent link="base_link"/>
+        <child link="${prefix}_WAIST"/>
+        <limit effort="1000" lower="-10" upper="10" velocity="1000"/>
+        <!-- joints rotates around the z-axis -->
+        <axis xyz="0 0 1"/>
+        <!-- placement of the joint -->
+        <origin xyz="0 0 ${base_2_WR_z}" rpy="0 0 0"/>
+        <!-- pybullet simulation parameters -->
+        <dynamics damping="0.0" friction="0.0"/>
+    </joint>
+    <link name="${prefix}_WAIST">
+        <inertial>
+            <!-- WAIST inertia -->
+            <mass value="0.73260731"/>
+            <origin xyz="-0.00013236 0.00599242 0.10576667" rpy="0 0 0"/>
+            <inertia ixx="0.10576667"
+                    ixy="0.00000024"
+                    ixz="-0.00000150"
+                    iyy="0.00138427"
+                    iyz="-0.00019152"
+                    izz="0.00249732"/>
+        </inertial>
+        <!-- WAIST LINK VISUAL -->
+        <visual>
+            <origin xyz="0 0 0" rpy="0 0 0"/>
+            <geometry>
+                <mesh filename="package://robot_properties_bolt/resources/meshes/${mesh_ext}/bolt_waist.${mesh_ext}"/>
+            </geometry>
+            <material name="${color_name}">
+                <color rgba="${color} ${opacity}"/>
+            </material>
+        </visual>
+        <!-- WAIST LINK COLLISION -->
+        <collision>
+            <origin xyz="0 0 0" rpy="0 0 0"/>
+            <geometry>
+                <mesh filename="package://robot_properties_bolt/resources/meshes/${mesh_ext}/bolt_waist.${mesh_ext}"/>
+            </geometry>
+            <material name="${color_name}">
+                <color rgba="${color} ${opacity}"/>
+            </material>
+        </collision>
+        <!-- Bullet specific paramters -->
+        <contact>
+            <lateral_friction value="1.0"/>
+            <restitution value="0.5"/>
+        </contact>
+    </link>
+    <joint name="${prefix}_SFE" type="revolute">
+        <parent link="${prefix}_WAIST"/>
+        <child link="${prefix}_ARM"/>
+        <limit effort="1000" lower="-10" upper="10" velocity="1000"/>
+        <!-- joints rotates around the y-axis -->
+        <axis xyz="0 1 0"/>
+        <!-- placement of the joint -->
+        <xacro:if value="${is_right}">
+            <origin xyz="0 ${-WR_2_SFE_y} ${WR_2_SFE_z}" rpy="0 0 0"/>
+        </xacro:if>
+        <xacro:unless value="${is_right}">
+            <origin xyz="0 ${WR_2_SFE_y} ${WR_2_SFE_z}" rpy="0 0 0"/>
+        </xacro:unless>
+        <!-- pybullet simulation parameters -->
+        <dynamics damping="0.0" friction="0.0"/>
+    </joint>
+    <link name="${prefix}_ARM">
+    <!-- ARM LINK INERTIAL -->
+        <xacro:unless value="${is_right}">
+        <!-- Left arm inertia -->
+            <inertial>
+                <mass value="0.12897855"/>
+                <origin xyz="0.02610170 0.01954144 -0.10554314" rpy="0 0 0"/>
+                <inertia ixx="0.00061875"
+                    ixy="0.00000154"
+                    ixz="-0.00027283"
+                    iyy="0.00081765"
+                    iyz="-0.00000622"
+                    izz="0.00020834"/>
+            </inertial>
+        </xacro:unless>
+        <xacro:if value="${is_right}">
+        <!-- Right arm inertia -->
+            <inertial>
+                <mass value="0.12897855"/>
+                <origin xyz="0.02610149 -0.01954144 -0.10554335" rpy="0 0 0"/>
+                <inertia ixx="0.00061875"
+                    ixy="-0.00000154"
+                    ixz="-0.00027283"
+                    iyy="0.00081765"
+                    iyz="0.00000622"
+                    izz="0.00020834"/>
+            </inertial>
+        </xacro:if>
+        <!-- ARM LINK VISUAL -->
+        <visual>
+            <origin xyz="0 0 0" rpy="0 0 0"/>
+            <geometry>
+                <xacro:unless value="${is_right}">
+                    <mesh filename="package://robot_properties_bolt/resources/meshes/${mesh_ext}/bolt_shoulder_fe_left_side.${mesh_ext}"/>
+                </xacro:unless>
+                <xacro:if value="${is_right}">
+                    <mesh filename="package://robot_properties_bolt/resources/meshes/${mesh_ext}/bolt_shoulder_fe_right_side.${mesh_ext}"/>
+                </xacro:if>
+            </geometry>
+            <material name="${color_name}">
+                <color rgba="${color} ${opacity}"/>
+            </material>
+        </visual>
+        <!-- ARM LINK COLLISION -->
+        <collision>
+            <origin xyz="0 0 0" rpy="0 0 0"/>
+            <geometry>
+                <xacro:unless value="${is_right}">
+                    <mesh filename="package://robot_properties_bolt/resources/meshes/${mesh_ext}/bolt_shoulder_fe_left_side.${mesh_ext}"/>
+                </xacro:unless>
+                <xacro:if value="${is_right}">
+                    <mesh filename="package://robot_properties_bolt/resources/meshes/${mesh_ext}/bolt_shoulder_fe_right_side.${mesh_ext}"/>
+                </xacro:if>
+            </geometry>
+            <material name="${color_name}">
+                <color rgba="${color} ${opacity}"/>
+            </material>
+        </collision>
+        <!-- Bullet specific paramters -->
+        <contact>
+            <lateral_friction value="0.0"/>
+            <restitution value="0.0"/>
+        </contact>
+    </link>
+    <!-- END ARM LINK -->
 </robot>
