Commit message: first version is ready

File: src/robot_properties_bolt/resources/xacro/bolt_humanoid.urdf.xacro (robot description, xacro)
@@ -13,4 +13,6 @@
   <!-- Include the legs -->
   <xacro:include filename="bolt.xacro"/>
+  <!-- Include the upper body -->
+  <xacro:include filename="upper_body.xacro"/>
   <!-- Include the fully parametrized bolt -->
   <xacro:bolt_full

File: src/robot_properties_bolt/resources/xacro/upper_body.xacro (robot description, xacro)
@@ -1,14 +1,15 @@
-<?xml version="1.0"?>
-<robot xmlns:xacro="http://playerstage.sourceforge.net/gazebo/xmlschema/#interface" name="bolt">
-  <!-- These are absolute distance value, the sign are decided below -->
+<?xml version="1.0" ?>
+<robot name="bolt"
+  xmlns:controller="http://playerstage.sourceforge.net/gazebo/xmlschema/#controller"
+  xmlns:interface="http://playerstage.sourceforge.net/gazebo/xmlschema/#interface"
+  xmlns:sensor="http://playerstage.sourceforge.net/gazebo/xmlschema/#sensor"
+  xmlns:xacro="http://playerstage.sourceforge.net/gazebo/xmlschema/#interface">
   <!-- WA stands for Waist Rotation joint, SFE is shoulder flexion-extension -->
   <xacro:property name="base_2_WR_z" value="${76.0 * 0.001}" />
-  <xacro:property name="WR_2_SFE_y" value="${110.0 * 0.001}" />
-  <xacro:property name="WR_2_SFE_z" value="${160.0 * 0.001}" />
-  <!-- Macro defining bolt upper_body. -->
-  <xacro:macro name="upper_body" params="prefix is_right has_side_motion mesh_ext color_name color">
-    <joint name="${prefix}_WR" type="revolute">
+  <xacro:macro name="upper_boddy" params="mesh_ext color_name color opacity">
+    <!-- wAIST link  -->
+    <joint name="WR" type="revolute">
         <parent link="base_link"/>
-        <child link="${prefix}_WAIST"/>
+        <child link="WAIST"/>
         <limit effort="1000" lower="-10" upper="10" velocity="1000"/>
         <!-- joints rotates around the z-axis -->
@@ -19,5 +20,5 @@
         <dynamics damping="0.0" friction="0.0"/>
     </joint>
-    <link name="${prefix}_WAIST">
+    <link name="WAIST">
         <inertial>
             <!-- WAIST inertia -->
@@ -53,88 +54,26 @@
         <!-- Bullet specific paramters -->
         <contact>
-            <lateral_friction value="1.0"/>
-            <restitution value="0.5"/>
+            <lateral_friction value=".0"/>
+            <restitution value="0."/>
         </contact>
     </link>
-    <joint name="${prefix}_SFE" type="revolute">
-        <parent link="${prefix}_WAIST"/>
-        <child link="${prefix}_ARM"/>
-        <limit effort="1000" lower="-10" upper="10" velocity="1000"/>
-        <!-- joints rotates around the y-axis -->
-        <axis xyz="0 1 0"/>
-        <!-- placement of the joint -->
-        <xacro:if value="${is_right}">
-            <origin xyz="0 ${-WR_2_SFE_y} ${WR_2_SFE_z}" rpy="0 0 0"/>
-        </xacro:if>
-        <xacro:unless value="${is_right}">
-            <origin xyz="0 ${WR_2_SFE_y} ${WR_2_SFE_z}" rpy="0 0 0"/>
-        </xacro:unless>
-        <!-- pybullet simulation parameters -->
-        <dynamics damping="0.0" friction="0.0"/>
-    </joint>
-    <link name="${prefix}_ARM">
-    <!-- ARM LINK INERTIAL -->
-        <xacro:unless value="${is_right}">
-        <!-- Left arm inertia -->
-            <inertial>
-                <mass value="0.12897855"/>
-                <origin xyz="0.02610170 0.01954144 -0.10554314" rpy="0 0 0"/>
-                <inertia ixx="0.00061875"
-                    ixy="0.00000154"
-                    ixz="-0.00027283"
-                    iyy="0.00081765"
-                    iyz="-0.00000622"
-                    izz="0.00020834"/>
-            </inertial>
-        </xacro:unless>
-        <xacro:if value="${is_right}">
-        <!-- Right arm inertia -->
-            <inertial>
-                <mass value="0.12897855"/>
-                <origin xyz="0.02610149 -0.01954144 -0.10554335" rpy="0 0 0"/>
-                <inertia ixx="0.00061875"
-                    ixy="-0.00000154"
-                    ixz="-0.00027283"
-                    iyy="0.00081765"
-                    iyz="0.00000622"
-                    izz="0.00020834"/>
-            </inertial>
-        </xacro:if>
-        <!-- ARM LINK VISUAL -->
-        <visual>
-            <origin xyz="0 0 0" rpy="0 0 0"/>
-            <geometry>
-                <xacro:unless value="${is_right}">
-                    <mesh filename="package://robot_properties_bolt/resources/meshes/${mesh_ext}/bolt_shoulder_fe_left_side.${mesh_ext}"/>
-                </xacro:unless>
-                <xacro:if value="${is_right}">
-                    <mesh filename="package://robot_properties_bolt/resources/meshes/${mesh_ext}/bolt_shoulder_fe_right_side.${mesh_ext}"/>
-                </xacro:if>
-            </geometry>
-            <material name="${color_name}">
-                <color rgba="${color} ${opacity}"/>
-            </material>
-        </visual>
-        <!-- ARM LINK COLLISION -->
-        <collision>
-            <origin xyz="0 0 0" rpy="0 0 0"/>
-            <geometry>
-                <xacro:unless value="${is_right}">
-                    <mesh filename="package://robot_properties_bolt/resources/meshes/${mesh_ext}/bolt_shoulder_fe_left_side.${mesh_ext}"/>
-                </xacro:unless>
-                <xacro:if value="${is_right}">
-                    <mesh filename="package://robot_properties_bolt/resources/meshes/${mesh_ext}/bolt_shoulder_fe_right_side.${mesh_ext}"/>
-                </xacro:if>
-            </geometry>
-            <material name="${color_name}">
-                <color rgba="${color} ${opacity}"/>
-            </material>
-        </collision>
-        <!-- Bullet specific paramters -->
-        <contact>
-            <lateral_friction value="0.0"/>
-            <restitution value="0.0"/>
-        </contact>
-    </link>
-    <!-- END ARM LINK -->
+    <!-- Include the arms -->
+    <xacro:include filename="arm.xacro"/>
+    <!-- Include the left arm -->
+    <xacro:arm
+        prefix="L"
+        is_right="false"
+        mesh_ext="${mesh_ext}"
+        color_name="${color_name}"
+        color="${color}"
+        opacity="${opacity}"/>
+    <!-- Include the right arm -->
+    <xacro:arm
+        prefix="R"
+        is_right="true"
+        mesh_ext="${mesh_ext}"
+        color_name="${color_name}"
+        color="${color}"
+        opacity="${opacity}"/>
+  </xacro:macro>
 </robot>
