Commit message: test humanoid demo, still has problem with upper body

File: src/robot_properties_bolt/resources/xacro/arm.xacro (robot description, xacro)
@@ -1,4 +1,4 @@
 <?xml version="1.0"?>
-<robot xmlns:xacro="http://playerstage.sourceforge.net/gazebo/xmlschema/#interface" name="bolt">
+<robot xmlns:xacro="http://playerstage.sourceforge.net/gazebo/xmlschema/#interface" name="bolt_humanoid">
   <!-- These are absolute distance value, the sign are decided below -->
   <!-- SFE is shoulder flexion-extension -->

File: src/robot_properties_bolt/resources/xacro/bolt_humanoid.urdf.xacro (robot description, xacro)
@@ -1,4 +1,4 @@
 <?xml version="1.0" ?>
-<robot name="bolt"
+<robot name="bolt_humanoid"
   xmlns:controller="http://playerstage.sourceforge.net/gazebo/xmlschema/#controller"
   xmlns:interface="http://playerstage.sourceforge.net/gazebo/xmlschema/#interface"
@@ -12,9 +12,7 @@
   <xacro:property name="has_passive_ankle" value="false" />
   <!-- Include the legs -->
-  <xacro:include filename="bolt.xacro"/>
-  <!-- Include the upper body -->
-  <xacro:include filename="upper_body.xacro"/>
+  <xacro:include filename="bolt_humanoid.xacro"/>
   <!-- Include the fully parametrized bolt -->
-  <xacro:bolt_full
+  <xacro:bolt_humanoid_full
       mesh_ext="${mesh_ext}"
       color_name="${color_name}"

File: src/robot_properties_bolt/resources/xacro/bolt_humanoid.xacro (robot description, xacro)
@@ -1,12 +1,11 @@
 <?xml version="1.0" ?>
-<robot name="bolt"
+<robot name="bolt_humanoid"
   xmlns:controller="http://playerstage.sourceforge.net/gazebo/xmlschema/#controller"
   xmlns:interface="http://playerstage.sourceforge.net/gazebo/xmlschema/#interface"
   xmlns:sensor="http://playerstage.sourceforge.net/gazebo/xmlschema/#sensor"
   xmlns:xacro="http://playerstage.sourceforge.net/gazebo/xmlschema/#interface">
-  <xacro:macro name="bolt_full" params="mesh_ext color_name color opacity new_leg has_passive_ankle">
-    <!-- This file is based on:  -->
+  <xacro:macro name="bolt_humanoid_full" params="mesh_ext color_name color opacity new_leg has_passive_ankle">
     <link name="base_link">
-      <!-- BASE LINK INERTIA -->
+      <!-- BASE LINK INERTIAL -->
       <inertial>
           <origin xyz="0 0 0" rpy="0 0 0" />
@@ -44,4 +43,12 @@
       </contact>
     </link> <!-- END BASE LINK -->
+    <!-- Include the upper body -->
+    <xacro:include filename="upper_body.xacro"/>
+    <!-- Include the upper body -->
+    <xacro:upper_body
+        mesh_ext="${mesh_ext}"
+        color_name="${color_name}"
+        color="${color}"
+        opacity="${opacity}"/>
     <!-- Include the legs -->
     <xacro:include filename="leg.xacro"/>

File: src/robot_properties_bolt/resources/xacro/upper_body.xacro (robot description, xacro)
@@ -1,12 +1,8 @@
 <?xml version="1.0" ?>
-<robot name="bolt"
-  xmlns:controller="http://playerstage.sourceforge.net/gazebo/xmlschema/#controller"
-  xmlns:interface="http://playerstage.sourceforge.net/gazebo/xmlschema/#interface"
-  xmlns:sensor="http://playerstage.sourceforge.net/gazebo/xmlschema/#sensor"
-  xmlns:xacro="http://playerstage.sourceforge.net/gazebo/xmlschema/#interface">
+<robot name="bolt_humanoid" xmlns:xacro="http://playerstage.sourceforge.net/gazebo/xmlschema/#interface">
   <!-- WA stands for Waist Rotation joint, SFE is shoulder flexion-extension -->
   <xacro:property name="base_2_WR_z" value="${76.0 * 0.001}" />
-  <xacro:macro name="upper_boddy" params="mesh_ext color_name color opacity">
-    <!-- wAIST link  -->
+  <xacro:macro name="upper_body" params="mesh_ext color_name color opacity">
+    <!-- WAIST link  -->
     <joint name="WR" type="revolute">
         <parent link="base_link"/>

Commit message: update stl files extensions

File: src/robot_properties_bolt/resources/xacro/arm.xacro (robot description, xacro)
@@ -58,6 +58,5 @@
                     <mesh filename="package://robot_properties_bolt/resources/meshes/${mesh_ext}/bolt_shoulder_fe_left_side.${mesh_ext}"/>
                 </xacro:unless>
-                <xacro:if value="${is_right}">
-                    <mesh filename="package://robot_properties_bolt/resources/meshes/${mesh_ext}/bolt_shoulder_fe_right_side.${mesh_ext}"/>
+                <xacro:if value="${is_right}">mesh filename="package://robot_properties_bolt/resources/meshes/${mesh_ext}/bolt_shoulder_fe_right_side.${mesh_ext}"/>
                 </xacro:if>
             </geometry>
@@ -88,3 +87,4 @@
     </link>
     <!-- END ARM LINK -->
+    </xacro:macro>
 </robot>

Commit message: visulization demos work

File: src/robot_properties_bolt/resources/xacro/arm.xacro (robot description, xacro)
@@ -8,5 +8,5 @@
   <xacro:macro name="arm" params="prefix is_right mesh_ext color_name color opacity">
     <joint name="${prefix}_SFE" type="revolute">
-        <parent link="${prefix}_WAIST"/>
+        <parent link="WAIST"/>
         <child link="${prefix}_ARM"/>
         <limit effort="1000" lower="-10" upper="10" velocity="1000"/>
@@ -58,5 +58,6 @@
                     <mesh filename="package://robot_properties_bolt/resources/meshes/${mesh_ext}/bolt_shoulder_fe_left_side.${mesh_ext}"/>
                 </xacro:unless>
-                <xacro:if value="${is_right}">mesh filename="package://robot_properties_bolt/resources/meshes/${mesh_ext}/bolt_shoulder_fe_right_side.${mesh_ext}"/>
+                <xacro:if value="${is_right}">
+                  <mesh filename="package://robot_properties_bolt/resources/meshes/${mesh_ext}/bolt_shoulder_fe_right_side.${mesh_ext}"/>
                 </xacro:if>
             </geometry>

Commit message: add the hand as an end-effector and change the name of waist to trunck

File: src/robot_properties_bolt/resources/xacro/arm.xacro (robot description, xacro)
@@ -3,10 +3,12 @@
   <!-- These are absolute distance value, the sign are decided below -->
   <!-- SFE is shoulder flexion-extension -->
-  <xacro:property name="WR_2_SFE_y" value="${110.0 * 0.001}" />
-  <xacro:property name="WR_2_SFE_z" value="${160.0 * 0.001}" />
+  <xacro:property name="TR_2_SFE_y" value="${110.0 * 0.001}" />
+  <xacro:property name="TR_2_SFE_z" value="${160.0 * 0.001}" />
+  <xacro:property name="SFE_2_WRIST_y" value="${20.0 * 0.001}" />
+  <xacro:property name="SFE_2_WRIST_z" value="${200.0 * 0.001}" />
   <!-- Macro defining bolt arm. -->
   <xacro:macro name="arm" params="prefix is_right mesh_ext color_name color opacity">
     <joint name="${prefix}_SFE" type="revolute">
-        <parent link="WAIST"/>
+        <parent link="TRUNK"/>
         <child link="${prefix}_ARM"/>
         <limit effort="1000" lower="-10" upper="10" velocity="1000"/>
@@ -15,8 +17,8 @@
         <!-- placement of the joint -->
         <xacro:if value="${is_right}">
-            <origin xyz="0 ${-WR_2_SFE_y} ${WR_2_SFE_z}" rpy="0 0 0"/>
+            <origin xyz="0 ${-TR_2_SFE_y} ${TR_2_SFE_z}" rpy="0 0 0"/>
         </xacro:if>
         <xacro:unless value="${is_right}">
-            <origin xyz="0 ${WR_2_SFE_y} ${WR_2_SFE_z}" rpy="0 0 0"/>
+            <origin xyz="0 ${TR_2_SFE_y} ${TR_2_SFE_z}" rpy="0 0 0"/>
         </xacro:unless>
         <!-- pybullet simulation parameters -->
@@ -88,4 +90,57 @@
     </link>
     <!-- END ARM LINK -->
-    </xacro:macro>
+    <!-- WRIST: Joint between the arm and the (dummy) hand -->
+    <joint name="${prefix}_WRIST" type="fixed">
+      <parent link="${prefix}_ARM"/>
+      <child link="${prefix}L_HAND"/>
+      <!-- Joint placement -->
+      <xacro:unless value="${is_right}">
+        <origin xyz="0 ${SFE_2_WRIST_y} ${-SFE_2_WRIST_z}" rpy="0 0 0" />
+      </xacro:unless>
+      <xacro:if value="${is_right}">
+        <origin xyz="0 ${-SFE_2_WRIST_y} ${-SFE_2_WRIST_z}" rpy="0 0 0" />
+      </xacro:if>
+      <!-- Limits (usefull?) -->
+      <limit effort="1000" lower="-10" upper="10" velocity="1000"/>
+      <!-- pybullet simulation parameters -->
+      <dynamics damping="0.0" friction="0.0"/>
+    </joint>
+    <link name="${prefix}_HAND">
+      <!-- HAND INERTIAL -->
+      <!-- This link is symmetrical left or right -->
+      <inertial>
+        <origin xyz="0 0 0.0" rpy="0 0 0" />
+        <mass value="0.0"/>
+        <inertia ixx="0.0" ixy="0.0" ixz="0.0"
+                           iyy="0.0" iyz="0.0"
+                                     izz="0.0"/>
+     </inertial>
+      <!-- HAND VISUAL -->
+      <visual>
+        <origin xyz="0 0 0" rpy="0 0 0" />
+        <geometry>
+          <mesh filename="package://robot_properties_bolt/resources/meshes/${mesh_ext}/with_foot/bolt_foot.${mesh_ext}"/>
+        </geometry>
+        <material name="${color_name}">
+            <color rgba="${color} ${opacity}"/>
+        </material>
+      </visual>
+      <!-- HAND COLLISION -->
+      <collision>
+        <origin xyz="0 0 0" rpy="0 0 0" />
+        <geometry>
+            <mesh filename="package://robot_properties_bolt/resources/meshes/${mesh_ext}/with_foot/bolt_foot.${mesh_ext}"/>
+        </geometry>
+        <material name="${color_name}">
+            <color rgba="${color} ${opacity}"/>
+        </material>
+      </collision>
+      <!-- Bullet specific paramters -->
+      <contact>
+        <lateral_friction value="1.0"/>
+        <restitution value="0.5"/>
+      </contact>
+    </link>
+    <!-- END HAND LINK -->
+  </xacro:macro>
 </robot>

File: src/robot_properties_bolt/resources/xacro/upper_body.xacro (robot description, xacro)
@@ -1,25 +1,25 @@
 <?xml version="1.0" ?>
 <robot name="bolt_humanoid" xmlns:xacro="http://playerstage.sourceforge.net/gazebo/xmlschema/#interface">
-  <!-- WA stands for Waist Rotation joint, SFE is shoulder flexion-extension -->
-  <xacro:property name="base_2_WR_z" value="${76.0 * 0.001}" />
+  <!-- WA stands for trunk Rotation joint, SFE is shoulder flexion-extension -->
+  <xacro:property name="base_2_TR_z" value="${76.0 * 0.001}" />
   <xacro:macro name="upper_body" params="mesh_ext color_name color opacity">
-    <!-- WAIST link  -->
-    <joint name="WR" type="revolute">
+    <!-- TRUNK link  -->
+    <joint name="TR" type="revolute">
         <parent link="base_link"/>
-        <child link="WAIST"/>
+        <child link="TRUNK"/>
         <limit effort="1000" lower="-10" upper="10" velocity="1000"/>
         <!-- joints rotates around the z-axis -->
         <axis xyz="0 0 1"/>
         <!-- placement of the joint -->
-        <origin xyz="0 0 ${base_2_WR_z}" rpy="0 0 0"/>
+        <origin xyz="0 0 ${base_2_TR_z}" rpy="0 0 0"/>
         <!-- pybullet simulation parameters -->
         <dynamics damping="0.0" friction="0.0"/>
     </joint>
-    <link name="WAIST">
+    <link name="TRUNK">
         <inertial>
-            <!-- WAIST inertia -->
+            <!-- TRUNK inertia -->
             <mass value="0.73260731"/>
             <origin xyz="-0.00013236 0.00599242 0.10576667" rpy="0 0 0"/>
-            <inertia ixx="0.10576667"
+            <inertia ixx="0.00371329"
                     ixy="0.00000024"
                     ixz="-0.00000150"
@@ -28,9 +28,9 @@
                     izz="0.00249732"/>
         </inertial>
-        <!-- WAIST LINK VISUAL -->
+        <!-- TRUNK LINK VISUAL -->
         <visual>
             <origin xyz="0 0 0" rpy="0 0 0"/>
             <geometry>
-                <mesh filename="package://robot_properties_bolt/resources/meshes/${mesh_ext}/bolt_waist.${mesh_ext}"/>
+                <mesh filename="package://robot_properties_bolt/resources/meshes/${mesh_ext}/bolt_trunk.${mesh_ext}"/>
             </geometry>
             <material name="${color_name}">
@@ -38,9 +38,9 @@
             </material>
         </visual>
-        <!-- WAIST LINK COLLISION -->
+        <!-- TRUNK LINK COLLISION -->
         <collision>
             <origin xyz="0 0 0" rpy="0 0 0"/>
             <geometry>
-                <mesh filename="package://robot_properties_bolt/resources/meshes/${mesh_ext}/bolt_waist.${mesh_ext}"/>
+                <mesh filename="package://robot_properties_bolt/resources/meshes/${mesh_ext}/bolt_trunk.${mesh_ext}"/>
             </geometry>
             <material name="${color_name}">

Commit message: debug the namings issues

File: src/robot_properties_bolt/resources/xacro/arm.xacro (robot description, xacro)
@@ -93,5 +93,5 @@
     <joint name="${prefix}_WRIST" type="fixed">
       <parent link="${prefix}_ARM"/>
-      <child link="${prefix}L_HAND"/>
+      <child link="${prefix}_HAND"/>
       <!-- Joint placement -->
       <xacro:unless value="${is_right}">
@@ -120,5 +120,5 @@
         <origin xyz="0 0 0" rpy="0 0 0" />
         <geometry>
-          <mesh filename="package://robot_properties_bolt/resources/meshes/${mesh_ext}/with_foot/bolt_foot.${mesh_ext}"/>
+          <mesh filename="package://robot_properties_bolt/resources/meshes/${mesh_ext}/bolt_foot.${mesh_ext}"/>
         </geometry>
         <material name="${color_name}">
@@ -130,5 +130,5 @@
         <origin xyz="0 0 0" rpy="0 0 0" />
         <geometry>
-            <mesh filename="package://robot_properties_bolt/resources/meshes/${mesh_ext}/with_foot/bolt_foot.${mesh_ext}"/>
+            <mesh filename="package://robot_properties_bolt/resources/meshes/${mesh_ext}/bolt_foot.${mesh_ext}"/>
         </geometry>
         <material name="${color_name}">

Commit message: update the length of the arm

File: src/robot_properties_bolt/resources/xacro/arm.xacro (robot description, xacro)
@@ -5,6 +5,6 @@
   <xacro:property name="TR_2_SFE_y" value="${110.0 * 0.001}" />
   <xacro:property name="TR_2_SFE_z" value="${160.0 * 0.001}" />
-  <xacro:property name="SFE_2_WRIST_y" value="${20.0 * 0.001}" />
-  <xacro:property name="SFE_2_WRIST_z" value="${200.0 * 0.001}" />
+  <xacro:property name="SFE_2_WRIST_x" value="${121 * 0.001}" />
+  <xacro:property name="SFE_2_WRIST_z" value="${210.0 * 0.001}" />
   <!-- Macro defining bolt arm. -->
   <xacro:macro name="arm" params="prefix is_right mesh_ext color_name color opacity">
@@ -96,8 +96,8 @@
       <!-- Joint placement -->
       <xacro:unless value="${is_right}">
-        <origin xyz="0 ${SFE_2_WRIST_y} ${-SFE_2_WRIST_z}" rpy="0 0 0" />
+        <origin xyz="${SFE_2_WRIST_x} 0 ${-SFE_2_WRIST_z}" rpy="0 0 0" />
       </xacro:unless>
       <xacro:if value="${is_right}">
-        <origin xyz="0 ${-SFE_2_WRIST_y} ${-SFE_2_WRIST_z}" rpy="0 0 0" />
+        <origin xyz="${-SFE_2_WRIST_x} 0 ${-SFE_2_WRIST_z}" rpy="0 0 0" />
       </xacro:if>
       <!-- Limits (usefull?) -->

Commit message: update the intial condition

File: src/robot_properties_bolt/resources/xacro/arm.xacro (robot description, xacro)
@@ -95,10 +95,5 @@
       <child link="${prefix}_HAND"/>
       <!-- Joint placement -->
-      <xacro:unless value="${is_right}">
-        <origin xyz="${SFE_2_WRIST_x} 0 ${-SFE_2_WRIST_z}" rpy="0 0 0" />
-      </xacro:unless>
-      <xacro:if value="${is_right}">
-        <origin xyz="${-SFE_2_WRIST_x} 0 ${-SFE_2_WRIST_z}" rpy="0 0 0" />
-      </xacro:if>
+      <origin xyz="${SFE_2_WRIST_x} 0 ${-SFE_2_WRIST_z}" rpy="0 0 0" />
       <!-- Limits (usefull?) -->
       <limit effort="1000" lower="-10" upper="10" velocity="1000"/>
